File: Hardware/Robosapien.kicad_pcb (KiCad board)
At the start: 2 copper layers, 59.2 x 45 mm, 76 parts, among them CN1 B2B-PH-K-S(LF)(SN), CN2 B2B-PH-K-S(LF)(SN), Q1 SS8050, Q2 SS8050, U1 ESP32-WROOM-32D(8MB), U2 CP2102-GMR, U3 BRCL3130ME, U4 TP4057, U5 TPS63020DSJR, U6 PCA9685PW,118, U7 PAM8303DBSC

Commit message: V2 Board
Parts:
- removed ? (x4): , 
- removed the C6 at (45.1, 27.4)
- removed the R12 at (42.8, 27.4)
- removed the R9 at (25.7, 25.7)
- removed the REF** at (65.0, 55.0)
- removed the REF** at (65.0, 58.0)
- removed the REF** at (67.0, 53.5)
- removed the REF** at (67.0, 55.0)
- removed the REF** at (67.0, 58.0)
- removed the REF** at (65.0, 56.5)
- removed the REF** at (67.0, 52.0)
- removed the REF** at (65.0, 52.0)
- removed the REF** at (67.0, 56.5)
- removed the REF** at (65.0, 53.5)
- removed U3: BRCL3130ME, easyeda2kicad:SOT-23-5_L2.9-W1.6-P0.95-LS2.8-BL
- added CN3: B2B-PH-K-S(LF)(SN), easyeda2kicad:CONN-TH_B2B-PH-K-S, F.Cu at (44.0, 29.9)
- added H8: Header 2.54 5P Female, easyeda2kicad:HDR-TH_5P-P2.54-V-F, F.Cu at (68.3, 51.7)
- added H9: Header 2.54 5P Female, easyeda2kicad:HDR-TH_5P-P2.54-V-F, F.Cu at (63.0, 57.0)
- added REF**: MountingHole_2.2mm_M2_Pad_Via, MountingHole:MountingHole_2.2mm_M2_Pad_Via, F.Cu at (22.4, 22.4)
- added REF**: MountingHole_2.2mm_M2_Pad_Via, MountingHole:MountingHole_2.2mm_M2_Pad_Via, F.Cu at (62.6, 22.4)
- added REF**: MountingHole_2.2mm_M2_Pad_Via, MountingHole:MountingHole_2.2mm_M2_Pad_Via, F.Cu at (22.4, 62.6)
- moved H4 2.06 mm to (77.0, 37.0)
- moved H5 2.06 mm to (74.4, 37.0)
- moved H7 2.06 mm to (79.5, 37.0)
- moved R17 2.06 mm to (78.1, 61.3)
- moved C21 2.06 mm to (80.3, 57.9)
- moved R16 2.06 mm to (76.0, 60.0)
- moved R18 2.06 mm to (79.0, 60.0)
- moved U7 2.06 mm to (74.8, 55.0)
- moved CN1 0.21 mm to (43.9, 25.1)
- renumbered C4 to C1, C13 to C10, C14 to C12, C3 to C13, C1 to C14, C2 to C15, C17 to C16, C21 to C17, C20 to C18, C18 to C19, C5 to C2, C19 to C20, C16 to C21, C8 to C3, C15 to C5, C12 to C6, C9 to C7, C7 to C8, C10 to C9, CN2 to CN1, CN1 to CN2, H3 to H1, H1 to H2, H4 to H3, H5 to H4, H7 to H5, H2 to H6, H6 to H7, R10 to R1, R1 to R11, R2 to R12, R5 to R13, R17 to R14, R18 to R15, R3 to R17, R4 to R18, R7 to R2, R6 to R3, R13 to R4, R8 to R5, R11 to R7, R14 to R8, R15 to R9, U4 to U1, U5 to U4, U1 to U5, U7 to U6, U6 to U7
Connections:
- CN1 pad 1: /BMS/BAT- -> GND
- CN1 pad 2: +BATT -> /BMS/BAT+
- U1 pad 3: +BATT -> /BMS/BAT+
Routing:
- net /BMS/BAT+: track 0.00 -> 13.6 mm
- net /BMS/BAT-: track 6.22 -> 0.00 mm
- net Net-(C6-Pad2): track 4.71 -> 0.00 mm
- net +BATT: track 147.1 -> 143.2 mm
- net /SDA: track 55.7 -> 58.2 mm
- net +3.3V: track 138.9 -> 140.5 mm
Other:
- board size 59.2 x 45 mm -> 99.1 x 50.1 mm
