File: Hardware/Robosapien.kicad_pcb (KiCad board)
At the start: 2 copper layers, 99.1 x 50.1 mm, 64 parts, among them CN1 B2B-PH-K-S(LF)(SN), CN2 B2B-PH-K-S(LF)(SN), CN3 B2B-PH-K-S(LF)(SN), Q1 SS8050, Q2 SS8050, U1 TP4057, U2 CP2102-GMR, U4 TPS63020DSJR, U5 ESP32-WROOM-32D(8MB), U6 PAM8303DBSC, U7 PCA9685PW,118

Commit message: PCB V2
Parts:
- removed C5, C6: 22uF, easyeda2kicad:C0603
- removed C7: 10uF, easyeda2kicad:C0402
- removed R9: 180kΩ 0603 75V, easyeda2kicad:R0603
- removed REF** (x3): MountingHole_2.2mm_M2_Pad_Via, MountingHole:MountingHole_2.2mm_M2_Pad_Via
- removed TV1: SRV05-4-P-T7 TVS, easyeda2kicad:SOT-23-6_L2.9-W1.6-P0.95-LS2.8-BR
- added C22: 10uF, easyeda2kicad:C0402, F.Cu at (-128.0, 8.50)
- added C23: 100uF, easyeda2kicad:CAP-SMD_L3.5-W2.8, F.Cu at (-124.1, 7.20)
- added C24: 100nF, easyeda2kicad:C0402_NEW, F.Cu at (-121.8, 8.70)
- added C25: 100nF, easyeda2kicad:C0402_NEW, F.Cu at (-102.7, 25.0)
- added C26: 100nF, easyeda2kicad:C0402_NEW, F.Cu at (-102.7, 27.6)
- added C27: 100uF 6.3V Tantal 3528, easyeda2kicad:CAP-SMD_L3.5-W2.8, F.Cu at (-99.2, 3.15)
- added C28: 16V 100nF X7R ±10% 0402, easyeda2kicad:C0402_NEW, F.Cu at (-105.1, 4.75)
- added C29: 22uF, easyeda2kicad:C0603, F.Cu at (-101.8, 14.6)
- added C30: 16V 100nF X7R ±10% 0402, easyeda2kicad:C0402_NEW, F.Cu at (-106.3, 4.75)
- added C31: 25V 1uF X5R ±10% 0402, easyeda2kicad:C0402, F.Cu at (-105.2, 2.15)
- added C32: 22uF, easyeda2kicad:C0603, F.Cu at (-100.1, 14.6)
- added C33: 100uF, easyeda2kicad:CAP-SMD_L3.5-W2.8, F.Cu at (-137.8, -2.75)
- added C34: 100uF, easyeda2kicad:CAP-SMD_L3.5-W2.8, F.Cu at (-110.7, -0.30)
- added C35: 100uF, easyeda2kicad:CAP-SMD_L3.5-W2.8, F.Cu at (-114.8, -10.8)
- added C36: 100uF, easyeda2kicad:CAP-SMD_L3.5-W2.8, F.Cu at (-132.3, -10.7)
- added C37: 100nF, easyeda2kicad:C0402_NEW, F.Cu at (-129.4, 26.1)
- added C4: 10uF, easyeda2kicad:C0402, F.Cu at (-97.8, 33.3)
- added D1: SMF05CT1G, easyeda2kicad:SOT-363_L2.0-W1.3-P0.65-LS2.1-BR, F.Cu at (-132.6, 31.4)
- added D10: SMF05CT1G, easyeda2kicad:SOT-363_L2.0-W1.3-P0.65-LS2.1-BR, F.Cu at (-122.6, -13.8)
- added D11: SS14, easyeda2kicad:SMA_L4.2-W2.6-LS5.3-RD, F.Cu at (-138.1, 16.1)
- added D12: SS14, easyeda2kicad:SMA_L4.2-W2.6-LS5.3-RD, F.Cu at (-135.2, 16.1)
- added D4: SMF05CT1G, easyeda2kicad:SOT-363_L2.0-W1.3-P0.65-LS2.1-BR, F.Cu at (-100.4, 17.8)
- added D5: SMF05CT1G, easyeda2kicad:SOT-363_L2.0-W1.3-P0.65-LS2.1-BR, F.Cu at (-106.9, -1.65)
- added D7: SMF05CT1G, easyeda2kicad:SOT-363_L2.0-W1.3-P0.65-LS2.1-BR, F.Cu at (-119.2, 3.40)
- added D8: SMF05CT1G, easyeda2kicad:SOT-363_L2.0-W1.3-P0.65-LS2.1-BR, F.Cu at (-127.7, 3.07)
- added D9: SMF05CT1G, easyeda2kicad:SOT-363_L2.0-W1.3-P0.65-LS2.1-BR, F.Cu at (-127.2, -13.8)
- added L3: 600Ω 200mA, easyeda2kicad:L0603, F.Cu at (-129.2, 24.6)
- added L4: 2.8A 1uH ±20% 45mΩ, easyeda2kicad:IND-SMD_L2.5-W2.0, F.Cu at (-130.8, 5.40)
- added L5: 120Ω 3A, easyeda2kicad:L1206, F.Cu at (-100.9, 31.6)
- added L6: 120Ω 3A, easyeda2kicad:L1206, F.Cu at (-103.2, 1.96)
- added L8: 120Ω 3A, easyeda2kicad:L1206, F.Cu at (-136.2, 11.0)
- added LED3: White Led 0603, easyeda2kicad:LED0603-R-RD_WHITE, F.Cu at (-124.9, 35.7)
- added LED4: White Led 0603, easyeda2kicad:LED0603-R-RD_WHITE, F.Cu at (-111.0, -19.9)
- added R10: 10kΩ 0402 50V, easyeda2kicad:R0402, F.Cu at (-100.2, 25.1)
- added R19: 10kΩ 0402 50V, easyeda2kicad:R0402, F.Cu at (-101.4, 25.1)
- added R20: 4.7kΩ 0402 50V, easyeda2kicad:R0402, F.Cu at (-109.3, -20.8)
- added R25: 4.7kΩ 0402 50V, easyeda2kicad:R0402, F.Cu at (-125.5, 33.9)
- C1: value 10uF -> 100nF; footprint easyeda2kicad:C0402 -> easyeda2kicad:C0402_NEW
- C10, C12: value 22uF -> 10uF; footprint easyeda2kicad:C0603 -> easyeda2kicad:C0402
- C13: value 25V 1uF X5R ±10% 0402 -> 22uF; footprint easyeda2kicad:C0402 -> easyeda2kicad:C0603
- C15: value 100nF -> 10uF; footprint easyeda2kicad:C0402_NEW -> easyeda2kicad:C0402
- C16: value 25V 1uF X5R ±10% 0402 -> 100nF; footprint easyeda2kicad:C0402 -> easyeda2kicad:C0402_NEW
- C2: value 1uF -> 10uF
- C21: value 6.3V 10uF X5R ±20% 0402 -> 22uF; footprint easyeda2kicad:C0402 -> easyeda2kicad:C0603
- C9: value 10uF -> 1uF
- L1: value 2.8A 1uH ±20% 45mΩ -> 120Ω 3A; footprint easyeda2kicad:IND-SMD_L2.5-W2.0 -> easyeda2kicad:L1206
- Q1, Q2: value SS8050 -> SS8050_C2150
- R2: value 1kΩ 0402 50V -> 100kΩ 0402 50V
- R3: value 47kΩ 0402 50V -> 10kΩ 0402 50V
- R8: value 1MΩ 0402 50V -> 18kΩ 0402 50V
- USB1: value USB Micro B 1.8A -> 10118193-0001LF; footprint easyeda2kicad:MICRO-USB-SMD_U254-051T-4BH23-S2S -> easyeda2kicad:MICRO-USB-SMD_10118193-0001LF
- moved H7 210.1 mm to (-123.7, -16.5), turned to 0 degrees
- moved H4 209.0 mm to (-123.7, -21.6), turned to 0 degrees
- moved H5 205.9 mm to (-123.7, -19.1), turned to 0 degrees
- moved C21 203.3 mm to (-110.3, -12.7), turned to 0 degrees
- moved R18 197.6 mm to (-110.6, 4.45), turned to 0 degrees
- moved R17 195.0 mm to (-108.5, 4.45)
- moved U7 193.0 mm to (-104.3, -16.8), turned to 0 degrees
- moved C12 192.4 mm to (-136.7, 8.55), turned to -90 degrees
- moved H6 192.0 mm to (-124.3, -2.15), turned to 0 degrees
- moved R16 191.8 mm to (-99.5, -17.6), turned to -90 degrees
- moved H2 189.0 mm to (-124.3, 0.40), turned to 0 degrees
- moved C10 188.5 mm to (-134.6, 8.50), turned to -90 degrees
- moved C11 187.6 mm to (-133.4, 8.50)
- moved H1 187.6 mm to (-124.3, -4.70), turned to 0 degrees
- moved H8 182.6 mm to (-105.4, -4.70), turned to 0 degrees
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Connections:
- net /CP2102/D+ renamed /USB_CP2102/D+
- net /CP2102/D- renamed /USB_CP2102/D-
- net /CP2102/RXD renamed /ESP_TX
- net /CP2102/TXD renamed /ESP_RX
- C1 pad 2: +3.3V -> Net-(U5-VDD33)
- C10 pad 2: +3.3V -> Net-(C10-Pad2)
- C11 pad 2: +BATT -> Net-(C10-Pad2)
- C12 pad 2: +3.3V -> Net-(D11-K)
- C13 pad 2: /CP2102/ESP_EN -> Net-(C13-Pad2)
- C16 pad 2: +BATT -> +3.3V
- C19 pad 2: +BATT -> Net-(U6-PVDD)
- C2 pad 2: Net-(C2-Pad2) -> +3.3V
- C8 pad 2: /BMS/Vin -> /VBUS
- C9 pad 2: +BATT -> +3.3V
- H1 pad 1: /SERVO1 -> +BATT
- H1 pad 2: /SERVO2 -> +BATT
- H1 pad 3: /SERVO3 -> +BATT
- H1 pad 4: /SERVO4 -> +BATT
- H1 pad 5: /SERVO5 -> +BATT
- H1 pad 6: /SERVO6 -> +BATT
- H1 pad 7: /SERVO7 -> +BATT
- H1 pad 8: /SERVO8 -> +BATT
- H1 pad 9: /SERVO9 -> +BATT
- H2 pad 1: +BATT -> /SERVO1
- H2 pad 2: +BATT -> /SERVO2
- H2 pad 3: +BATT -> /SERVO3
- H2 pad 4: +BATT -> /SERVO4
- H2 pad 5: +BATT -> /SERVO5
- H2 pad 6: +BATT -> /SERVO6
- H2 pad 7: +BATT -> /SERVO7
- H2 pad 8: +BATT -> /SERVO8
- H2 pad 9: +BATT -> /SERVO9
- H5 pad 1: /Servo Extender/SERVO1 -> GND
- H5 pad 2: /Servo Extender/SERVO2 -> GND
- H5 pad 3: /Servo Extender/SERVO3 -> GND
- H5 pad 4: /Servo Extender/SERVO4 -> GND
- H5 pad 5: /Servo Extender/SERVO5 -> GND
- H5 pad 6: /Servo Extender/SERVO6 -> GND
- H5 pad 7: /Servo Extender/SERVO7 -> GND
- H5 pad 8: /Servo Extender/SERVO8 -> GND
- H5 pad 9: /Servo Extender/SERVO9 -> GND
- H7 pad 1: GND -> /Servo Extender/SERVO9
- H7 pad 2: GND -> /Servo Extender/SERVO8
- H7 pad 3: GND -> /Servo Extender/SERVO7
- H7 pad 4: GND -> /Servo Extender/SERVO6
- H7 pad 5: GND -> /Servo Extender/SERVO5
- H7 pad 6: GND -> /Servo Extender/SERVO4
- H7 pad 7: GND -> /Servo Extender/SERVO3
- H7 pad 8: GND -> /Servo Extender/SERVO2
- H7 pad 9: GND -> /Servo Extender/SERVO1
- L1 pad 1: Net-(L1-Pad1) -> +3.3V
- L1 pad 2: Net-(L1-Pad2) -> Net-(C13-Pad2)
- Q1 pad 1: Net-(Q1-Pad1) -> Net-(Q1-B)
- Q1 pad 2: /CP2102/RTS -> /USB_CP2102/RTS
- Q1 pad 3: /CP2102/ESP_EN -> /ESP_EN
- Q2 pad 1: Net-(Q2-Pad1) -> Net-(Q2-B)
- Q2 pad 2: /CP2102/DTR -> /USB_CP2102/DTR
- Q2 pad 3: /CP2102/ESP_IO0 -> /ESP_IO0
- R1 pad 1: /CP2102/RTS -> /ESP_IO0
- R1 pad 2: Net-(Q2-Pad1) -> +3.3V
- R13 pad 2: /CP2102/ESP_EN -> /ESP_EN
- R2 pad 1: +3.3V -> Net-(U4-FB)
- R2 pad 2: Net-(R2-Pad2) -> Net-(C13-Pad2)
- R3 pad 1: /BMS/Vin -> /USB_CP2102/DTR
- R3 pad 2: Net-(C2-Pad2) -> Net-(Q1-B)
- R5 pad 1: /CP2102/DTR -> /USB_CP2102/RTS
- R5 pad 2: Net-(Q1-Pad1) -> Net-(Q2-B)
- R7 pad 2: /BMS/Vin -> /VBUS
- R8 pad 1: Net-(R8-Pad1) -> GND
- R8 pad 2: +3.3V -> Net-(U4-FB)
- U1 pad 4: /BMS/Vin -> /VBUS
- U2 pad 24: /CP2102/RTS -> /USB_CP2102/RTS
- U2 pad 28: /CP2102/DTR -> /USB_CP2102/DTR
- U2 pad 6: +3.3V -> Net-(U2-REGIN)
- U2 pad 7: +3.3V -> Net-(U2-REGIN)
- U2 pad 8: Net-(C2-Pad2) -> /VBUS
- U2 pad 9: Net-(R2-Pad2) -> unconnected-(U2-~{RST}-Pad9)
- U4 pad 10: +BATT -> Net-(C10-Pad2)
- U4 pad 11: +BATT -> Net-(C10-Pad2)
- U4 pad 3: Net-(R8-Pad1) -> Net-(U4-FB)
- U4 pad 4: +3.3V -> Net-(C13-Pad2)
- U4 pad 5: +3.3V -> Net-(C13-Pad2)
- U4 pad 6: Net-(L1-Pad2) -> Net-(L4-Pad2)
- U4 pad 7: Net-(L1-Pad2) -> Net-(L4-Pad2)
- U4 pad 8: Net-(L1-Pad1) -> Net-(L4-Pad1)
- U4 pad 9: Net-(L1-Pad1) -> Net-(L4-Pad1)
- U5 pad 2: +3.3V -> Net-(U5-VDD33)
- U5 pad 25: /CP2102/ESP_IO0 -> /ESP_IO0
- U5 pad 3: /CP2102/ESP_EN -> /ESP_EN
- U6 pad 2: +BATT -> Net-(U6-PVDD)
- U6 pad 3: +BATT -> Net-(U6-PVDD)
- U7 pad 1: GND -> +3.3V
- U7 pad 2: GND -> +3.3V
- U7 pad 3: GND -> +3.3V
- U7 pad 4: GND -> +3.3V
- U7 pad 5: GND -> +3.3V
- USB1 pad 1: /BMS/Vin -> /VBUS
Routing:
- net +3.3V: track 140.5 -> 53.3 mm, vias 5 -> 15
- net /VBUS: track 0.00 -> 69.1 mm, vias 0 -> 2
- net GND: track 0.00 -> 61.8 mm, vias 25 -> 99
- net /Screen3: track 6.08 -> 47.0 mm, vias 0 -> 1
- net /ESP_EN: track 0.00 -> 38.0 mm, vias 0 -> 3
- net /BMS/Vin: track 30.9 -> 0.00 mm, vias 3 -> 0
- net /ESP_IO0: track 0.00 -> 27.2 mm, vias 0 -> 2
- net /CP2102/ESP_EN: track 27.1 -> 0.00 mm, vias 2 -> 0
- net /Screen4: track 9.01 -> 32.0 mm, vias 0 -> 2
- net /Screen1: track 6.08 -> 27.1 mm, vias 0 -> 1
- net +BATT: track 143.2 -> 122.7 mm, vias 0 -> 16
- net /CP2102/ESP_IO0: track 19.7 -> 0.00 mm, vias 2 -> 0
- net /Servo Extender/SERVO8: track 24.1 -> 41.9 mm
- net /Servo Extender/SERVO1: track 5.23 -> 20.8 mm
- net /USB_CP2102/RTS: track 0.00 -> 12.1 mm
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- added copper zone on F.Cu, net +3.3V
- added copper zone on In2.Cu, net +3.3V
- added copper zone on In2.Cu, net +BATT
- added copper zone on In1.Cu, net GND
- added copper zone on F.Cu, net Net-(C10-Pad2)
- added copper zone on F.Cu, net Net-(C13-Pad2)
- added copper zone on F.Cu, net Net-(L4-Pad1)
- added copper zone on F.Cu, net Net-(L4-Pad2)
- added copper zone on F.Cu, net Net-(U6-PVDD)
Other:
- board size 99.1 x 50.1 mm -> 45 x 61 mm
- copper layers 2 -> 4
- board text removed: "+BAT-"
- board text removed: "- + Screen"
- board text removed: "1 2 3 .. Servo"
- board text removed: "9 8 7 .. Servo"
- board text removed: "S + -"
- board text removed: "Speaker - +"

Commit message: adsads
Parts:
- removed C16: 100nF, easyeda2kicad:C0402_NEW
- removed C21: 22uF, easyeda2kicad:C0603
- removed C35, C36: 100uF, easyeda2kicad:CAP-SMD_L3.5-W2.8
- removed D10, D9: SMF05CT1G, easyeda2kicad:SOT-363_L2.0-W1.3-P0.65-LS2.1-BR
- removed H4, H5, H7: 9P 2.54 Male Header, easyeda2kicad:HDR-TH_9P-P2.54-V-M
- removed H9: Header 2.54 5P Female, easyeda2kicad:HDR-TH_5P-P2.54-V-F
- removed LED4: White Led 0603, easyeda2kicad:LED0603-R-RD_WHITE
- removed R16: 10kΩ 0402 50V, easyeda2kicad:R0402
- removed R20: 4.7kΩ 0402 50V, easyeda2kicad:R0402
- removed U7: PCA9685PW,118, easyeda2kicad:TSSOP-28_L9.7-W4.4-P0.65-LS6.4-TL
Routing:
- net /Servo Extender/SERVO8: track 41.9 -> 0.00 mm
- net /Servo Extender/SERVO9: track 37.4 -> 0.00 mm, vias 2 -> 0
- net +3.3V: track 53.3 -> 18.6 mm, vias 15 -> 13
- net /Servo Extender/SERVO7: track 25.8 -> 0.00 mm
- net /Servo Extender/SERVO5: track 23.3 -> 0.00 mm
- net /Servo Extender/SERVO6: track 23.3 -> 0.00 mm
- net /Servo Extender/SERVO1: track 20.8 -> 0.00 mm
- net +BATT: track 122.7 -> 104.4 mm, vias 16 -> 9
- net /Servo Extender/SERVO2: track 17.0 -> 0.00 mm
- net /Servo Extender/SERVO3: track 16.9 -> 0.00 mm, vias 1 -> 0
- net /Servo Extender/SERVO4: track 16.7 -> 0.00 mm, vias 1 -> 0
- net /SDA: track 55.4 -> 42.8 mm
- net /SCL: track 61.0 -> 49.5 mm
- net GND: track 61.8 -> 55.7 mm, vias 99 -> 87
- net Net-(U7-~{OE}): track 1.94 -> 0.00 mm
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Other:
- board size 45 x 61 mm -> 45 x 45 mm
