File: Hardware/cp2102.kicad_sch (KiCad schematic)
At the start: 8 parts

Commit message: Added esp32 and bms
Parts:
- added Q? (x2): SS8050, easyeda2kicad:SOT-23-3_L2.9-W1.3-P1.90-LS2.4-BR, symbol easyeda2kicad:SS8050_C2150
- added R? (x2): 10kΩ 0402 50V, easyeda2kicad:R0402, symbol easyeda2kicad:10kΩ 0402 50V
Connections:
- net RTS: now reaches U?.24 (RTS)
- net RTS: now also Q?.2 (E), R?.1
- net RXD: now reaches U?.25 (RXD)
- net TXD: now reaches U?.26 (TXD)
- net DTR: now reaches U?.28 (DTR)
- net DTR: now also Q?.2 (E), R?.1
- new net: Q?.1 (B), R?.2 (x2)
- new net ESP_EN: Q?.3 (C)
- new net ESP_IO0: Q?.3 (C)
- no-connect marks 18 -> 20
Other:
- note added: "Esp32 Boot Mode Logic"
Changed lines of the file:
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@@
   (no_connect (at 174.625 108.585))
   (no_connect (at 149.225 80.645))
+  (no_connect (at 177.165 62.865))
   (no_connect (at 50.165 65.405))
   (no_connect (at 194.945 80.645))
+  (no_connect (at 167.005 62.865))
   (no_connect (at 65.405 106.68))
   (no_connect (at 194.945 85.725))
@@
     (stroke (width 0) (type default) (color 0 0 0 0))
   )
+  (wire (pts (xy 239.395 122.555) (xy 217.805 122.555))
+    (stroke (width 0) (type default) (color 0 0 0 0))
+  )
   (wire (pts (xy 164.465 108.585) (xy 164.465 113.03))
     (stroke (width 0) (type default) (color 0 0 0 0))
   )
+  (wire (pts (xy 239.395 118.745) (xy 219.71 118.745))
+    (stroke (width 0) (type default) (color 0 0 0 0))
+  )
+  (wire (pts (xy 217.805 122.555) (xy 217.805 113.665))
+    (stroke (width 0) (type default) (color 0 0 0 0))
+  )
   (wire (pts (xy 164.465 113.03) (xy 132.08 113.03))
     (stroke (width 0) (type default) (color 0 0 0 0))
@@
     (stroke (width 0) (type default) (color 0 0 0 0))
   )
+  (wire (pts (xy 219.71 127.635) (xy 224.155 127.635))
+    (stroke (width 0) (type default) (color 0 0 0 0))
+  )
   (wire (pts (xy 75.565 57.785) (xy 75.565 73.66))
     (stroke (width 0) (type default) (color 0 0 0 0))
@@
     (stroke (width 0) (type default) (color 0 0 0 0))
   )
+  (wire (pts (xy 217.805 113.665) (xy 224.155 113.665))
+    (stroke (width 0) (type default) (color 0 0 0 0))
+  )
+  (wire (pts (xy 219.71 118.745) (xy 219.71 127.635))
+    (stroke (width 0) (type default) (color 0 0 0 0))
+  )
   (wire (pts (xy 65.405 62.865) (xy 92.075 62.865))
     (stroke (width 0) (type default) (color 0 0 0 0))
+  )
+  (text "Esp32 Boot Mode Logic" (at 213.995 104.775 0)
+    (effects (font (size 1.27 1.27)) (justify left bottom))
+  )
+  (label "RTS" (at 174.625 62.865 90)
+    (effects (font (size 1.27 1.27)) (justify left bottom))
+  )
+  (label "RTS" (at 219.71 127.635 180)
+    (effects (font (size 1.27 1.27)) (justify right bottom))
+  )
+  (label "DTR" (at 217.805 113.665 180)
+    (effects (font (size 1.27 1.27)) (justify right bottom))
   )
   (label "VBUS" (at 92.075 57.785 0)
@@
     (effects (font (size 1.27 1.27)) (justify left bottom))
   )
+  (label "DTR" (at 164.465 62.865 90)
+    (effects (font (size 1.27 1.27)) (justify left bottom))
+  )
   (label "D+" (at 149.225 85.725 180)
     (effects (font (size 1.27 1.27)) (justify right bottom))
@@
     (effects (font (size 1.27 1.27)) (justify left bottom))
   )
+  (hierarchical_label "ESP_EN" (shape tri_state) (at 239.395 108.585 0)
+    (effects (font (size 1.27 1.27)) (justify left))
+  )
+  (hierarchical_label "VBUS" (shape input) (at 75.565 57.785 90)
+    (effects (font (size 1.27 1.27)) (justify left))
+  )
+  (hierarchical_label "ESP_IO0" (shape tri_state) (at 239.395 132.715 0)
+    (effects (font (size 1.27 1.27)) (justify left))
+  )
+  (hierarchical_label "TXD" (shape input) (at 169.545 62.865 90)
+    (effects (font (size 1.27 1.27)) (justify left))
+  )
+  (hierarchical_label "RXD" (shape input) (at 172.085 62.865 90)
+    (effects (font (size 1.27 1.27)) (justify left))
+  )
+  (symbol (lib_id "easyeda2kicad:10kΩ 0402 50V") (at 229.235 113.665 0) (unit 1)
+    (in_bom yes) (on_board yes) (fields_autoplaced)
+    (property "Reference" "R?" (id 0) (at 229.235 107.315 0))
+    (property "Value" "10kΩ 0402 50V" (id 1) (at 229.235 109.855 0))
+    (property "Footprint" "easyeda2kicad:R0402" (id 2) (at 229.235 121.285 0)
+      (effects (font (size 1.27 1.27)) hide)
+    )
+    (property "Datasheet" "https://lcsc.com/product-detail/Chip-Resistor-Surface-Mount-UniOhm_10KR-1002-1_C25744.html" (id 3) (at 229.235 123.825 0)
+      (effects (font (size 1.27 1.27)) hide)
+    )
+    (property "Manufacturer" "UNI-ROYAL(厚声)" (id 4) (at 229.235 126.365 0)
+      (effects (font (size 1.27 1.27)) hide)
+    )
+    (property "LCSC Part" "C25744" (id 5) (at 229.235 128.905 0)
+      (effects (font (size 1.27 1.27)) hide)
+    )
+    (property "JLC Part" "Basic Part" (id 6) (at 229.235 131.445 0)
+      (effects (font (size 1.27 1.27)) hide)
+    )
+    (pin "1")
+    (pin "2")
+  )
   (symbol (lib_id "easyeda2kicad:25V 1uF X5R ±10% 0402") (at 132.08 118.11 90) (unit 1)
     (in_bom yes) (on_board yes) (fields_autoplaced)
@@
     )
     (pin "1")
+  )
+  (symbol (lib_id "easyeda2kicad:SS8050_C2150") (at 239.395 113.665 0) (unit 1)
+    (in_bom yes) (on_board yes)
+    (property "Reference" "Q?" (id 0) (at 243.205 112.395 0)
+      (effects (font (size 1.27 1.27)) (justify left))
+    )
+    (property "Value" "SS8050" (id 1) (at 243.205 114.935 0)
+      (effects (font (size 1.27 1.27)) (justify left))
+    )
+    (property "Footprint" "easyeda2kicad:SOT-23-3_L2.9-W1.3-P1.90-LS2.4-BR" (id 2) (at 239.395 126.365 0)
+      (effects (font (size 1.27 1.27)) hide)
+    )
+    (property "Datasheet" "https://lcsc.com/product-detail/Transistors-NPN-PNP_SS8050-Y1-200-350_C2150.html" (id 3) (at 239.395 128.905 0)
+      (effects (font (size 1.27 1.27)) hide)
+    )
+    (property "Manufacturer" "CJ(江苏长电/长晶)" (id 4) (at 239.395 131.445 0)
+      (effects (font (size 1.27 1.27)) hide)
+    )
+    (property "LCSC Part" "C2150" (id 5) (at 239.395 133.985 0)
+      (effects (font (size 1.27 1.27)) hide)
+    )
+    (property "JLC Part" "Basic Part" (id 6) (at 239.395 136.525 0)
+      (effects (font (size 1.27 1.27)) hide)
+    )
+    (pin "1")
+    (pin "2")
+    (pin "3")
   )
   (symbol (lib_id "easyeda2kicad:22kΩ 0402 50V") (at 127.635 118.11 90) (unit 1)
@@
     (pin "1")
   )
+  (symbol (lib_id "easyeda2kicad:10kΩ 0402 50V") (at 229.235 127.635 0) (unit 1)
+    (in_bom yes) (on_board yes) (fields_autoplaced)
+    (property "Reference" "R?" (id 0) (at 229.235 121.285 0))
+    (property "Value" "10kΩ 0402 50V" (id 1) (at 229.235 123.825 0))
+    (property "Footprint" "easyeda2kicad:R0402" (id 2) (at 229.235 135.255 0)
+      (effects (font (size 1.27 1.27)) hide)
+    )
+    (property "Datasheet" "https://lcsc.com/product-detail/Chip-Resistor-Surface-Mount-UniOhm_10KR-1002-1_C25744.html" (id 3) (at 229.235 137.795 0)
+      (effects (font (size 1.27 1.27)) hide)
+    )
+    (property "Manufacturer" "UNI-ROYAL(厚声)" (id 4) (at 229.235 140.335 0)
+      (effects (font (size 1.27 1.27)) hide)
+    )
+    (property "LCSC Part" "C25744" (id 5) (at 229.235 142.875 0)
+      (effects (font (size 1.27 1.27)) hide)
+    )
+    (property "JLC Part" "Basic Part" (id 6) (at 229.235 145.415 0)
+      (effects (font (size 1.27 1.27)) hide)
+    )
+    (pin "1")
+    (pin "2")
+  )
   (symbol (lib_id "power:GND") (at 132.08 123.19 0) (unit 1)
     (in_bom yes) (on_board yes) (fields_autoplaced)
@@
     (pin "1")
   )
+  (symbol (lib_id "easyeda2kicad:SS8050_C2150") (at 239.395 127.635 0) (mirror x) (unit 1)
+    (in_bom yes) (on_board yes)
+    (property "Reference" "Q?" (id 0) (at 243.205 128.905 0)
+      (effects (font (size 1.27 1.27)) (justify left))
+    )
+    (property "Value" "SS8050" (id 1) (at 243.205 126.365 0)
+      (effects (font (size 1.27 1.27)) (justify left))
+    )
+    (property "Footprint" "easyeda2kicad:SOT-23-3_L2.9-W1.3-P1.90-LS2.4-BR" (id 2) (at 239.395 114.935 0)
+      (effects (font (size 1.27 1.27)) hide)
+    )
+    (property "Datasheet" "https://lcsc.com/product-detail/Transistors-NPN-PNP_SS8050-Y1-200-350_C2150.html" (id 3) (at 239.395 112.395 0)
+      (effects (font (size 1.27 1.27)) hide)
+    )
+    (property "Manufacturer" "CJ(江苏长电/长晶)" (id 4) (at 239.395 109.855 0)
+      (effects (font (size 1.27 1.27)) hide)
+    )
+    (property "LCSC Part" "C2150" (id 5) (at 239.395 107.315 0)
+      (effects (font (size 1.27 1.27)) hide)
+    )
+    (property "JLC Part" "Basic Part" (id 6) (at 239.395 104.775 0)
+      (effects (font (size 1.27 1.27)) hide)
+    )
+    (pin "1")
+    (pin "2")
+    (pin "3")
+  )
   (symbol (lib_id "easyeda2kicad:47kΩ 0402 50V") (at 122.555 113.03 0) (unit 1)

Commit message: New pcb
Parts:
- gave numbers to parts that had none: 12
Changed lines of the file:
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@@
   (symbol (lib_id "easyeda2kicad:10kΩ 0402 50V") (at 229.235 113.665 0) (unit 1)
     (in_bom yes) (on_board yes) (fields_autoplaced)
-    (property "Reference" "R?" (id 0) (at 229.235 107.315 0))
+    (property "Reference" "R8" (id 0) (at 229.235 107.315 0))
     (property "Value" "10kΩ 0402 50V" (id 1) (at 229.235 109.855 0))
     (property "Footprint" "easyeda2kicad:R0402" (id 2) (at 229.235 121.285 0)
@@
   (symbol (lib_id "easyeda2kicad:25V 1uF X5R ±10% 0402") (at 132.08 118.11 90) (unit 1)
     (in_bom yes) (on_board yes) (fields_autoplaced)
-    (property "Reference" "C?" (id 0) (at 135.89 116.8399 90)
+    (property "Reference" "C5" (id 0) (at 135.89 116.8399 90)
       (effects (font (size 1.27 1.27)) (justify right))
     )
@@
   (symbol (lib_id "power:+3.3V") (at 167.005 118.745 180) (unit 1)
     (in_bom yes) (on_board yes) (fields_autoplaced)
-    (property "Reference" "#PWR?" (id 0) (at 167.005 114.935 0)
+    (property "Reference" "#PWR031" (id 0) (at 167.005 114.935 0)
       (effects (font (size 1.27 1.27)) hide)
     )
@@
   (symbol (lib_id "easyeda2kicad:SS8050_C2150") (at 239.395 113.665 0) (unit 1)
     (in_bom yes) (on_board yes)
-    (property "Reference" "Q?" (id 0) (at 243.205 112.395 0)
+    (property "Reference" "Q1" (id 0) (at 243.205 112.395 0)
       (effects (font (size 1.27 1.27)) (justify left))
     )
@@
   (symbol (lib_id "easyeda2kicad:22kΩ 0402 50V") (at 127.635 118.11 90) (unit 1)
     (in_bom yes) (on_board yes)
-    (property "Reference" "R?" (id 0) (at 123.19 116.84 90)
+    (property "Reference" "R9" (id 0) (at 123.19 116.84 90)
       (effects (font (size 1.27 1.27)) (justify right))
     )
@@
   (symbol (lib_id "easyeda2kicad:SRV05-4-P-T7 TVS") (at 76.835 90.17 270) (unit 1)
     (in_bom yes) (on_board yes) (fields_autoplaced)
-    (property "Reference" "TV?" (id 0) (at 95.25 88.8999 90)
+    (property "Reference" "TV1" (id 0) (at 95.25 88.8999 90)
       (effects (font (size 1.27 1.27)) (justify left))
     )
@@
   (symbol (lib_id "power:GND") (at 127.635 123.19 0) (unit 1)
     (in_bom yes) (on_board yes) (fields_autoplaced)
-    (property "Reference" "#PWR?" (id 0) (at 127.635 129.54 0)
+    (property "Reference" "#PWR032" (id 0) (at 127.635 129.54 0)
       (effects (font (size 1.27 1.27)) hide)
     )
@@
   (symbol (lib_id "easyeda2kicad:USB Micro B 1.8A") (at 40.005 62.865 0) (unit 1)
     (in_bom yes) (on_board yes) (fields_autoplaced)
-    (property "Reference" "USB?" (id 0) (at 38.735 46.99 0))
+    (property "Reference" "USB1" (id 0) (at 38.735 46.99 0))
     (property "Value" "USB Micro B 1.8A" (id 1) (at 38.735 49.53 0))
     (property "Footprint" "easyeda2kicad:MICRO-USB-SMD_U254-051T-4BH23-S2S" (id 2) (at 40.005 75.565 0)
@@
   (symbol (lib_id "power:GND") (at 27.305 62.865 270) (unit 1)
     (in_bom yes) (on_board yes) (fields_autoplaced)
-    (property "Reference" "#PWR?" (id 0) (at 20.955 62.865 0)
+    (property "Reference" "#PWR022" (id 0) (at 20.955 62.865 0)
       (effects (font (size 1.27 1.27)) hide)
     )
@@
   (symbol (lib_id "power:GND") (at 50.165 67.945 90) (unit 1)
     (in_bom yes) (on_board yes) (fields_autoplaced)
-    (property "Reference" "#PWR?" (id 0) (at 56.515 67.945 0)
+    (property "Reference" "#PWR024" (id 0) (at 56.515 67.945 0)
       (effects (font (size 1.27 1.27)) hide)
     )
@@
   (symbol (lib_id "easyeda2kicad:1kΩ 0402 50V") (at 167.005 113.665 90) (unit 1)
     (in_bom yes) (on_board yes) (fields_autoplaced)
-    (property "Reference" "R?" (id 0) (at 168.91 112.3949 90)
+    (property "Reference" "R7" (id 0) (at 168.91 112.3949 90)
       (effects (font (size 1.27 1.27)) (justify right))
     )
@@
   (symbol (lib_id "power:GND") (at 161.925 62.865 180) (unit 1)
     (in_bom yes) (on_board yes) (fields_autoplaced)
-    (property "Reference" "#PWR?" (id 0) (at 161.925 56.515 0)
+    (property "Reference" "#PWR023" (id 0) (at 161.925 56.515 0)
       (effects (font (size 1.27 1.27)) hide)
     )
@@
   (symbol (lib_id "easyeda2kicad:10kΩ 0402 50V") (at 229.235 127.635 0) (unit 1)
     (in_bom yes) (on_board yes) (fields_autoplaced)
-    (property "Reference" "R?" (id 0) (at 229.235 121.285 0))
+    (property "Reference" "R10" (id 0) (at 229.235 121.285 0))
     (property "Value" "10kΩ 0402 50V" (id 1) (at 229.235 123.825 0))
     (property "Footprint" "easyeda2kicad:R0402" (id 2) (at 229.235 135.255 0)
@@
   (symbol (lib_id "power:GND") (at 132.08 123.19 0) (unit 1)
     (in_bom yes) (on_board yes) (fields_autoplaced)
-    (property "Reference" "#PWR?" (id 0) (at 132.08 129.54 0)
+    (property "Reference" "#PWR033" (id 0) (at 132.08 129.54 0)
       (effects (font (size 1.27 1.27)) hide)
     )
@@
   (symbol (lib_id "power:GND") (at 75.565 106.68 0) (unit 1)
     (in_bom yes) (on_board yes) (fields_autoplaced)
-    (property "Reference" "#PWR?" (id 0) (at 75.565 113.03 0)
+    (property "Reference" "#PWR030" (id 0) (at 75.565 113.03 0)
       (effects (font (size 1.27 1.27)) hide)
     )
@@
   (symbol (lib_id "power:GND") (at 135.89 100.965 0) (unit 1)
     (in_bom yes) (on_board yes) (fields_autoplaced)
-    (property "Reference" "#PWR?" (id 0) (at 135.89 107.315 0)
+    (property "Reference" "#PWR029" (id 0) (at 135.89 107.315 0)
       (effects (font (size 1.27 1.27)) hide)
     )
@@
   (symbol (lib_id "power:+3.3V") (at 135.89 93.345 0) (unit 1)
     (in_bom yes) (on_board yes)
-    (property "Reference" "#PWR?" (id 0) (at 135.89 97.155 0)
+    (property "Reference" "#PWR027" (id 0) (at 135.89 97.155 0)
       (effects (font (size 1.27 1.27)) hide)
     )
@@
   (symbol (lib_id "easyeda2kicad:SS8050_C2150") (at 239.395 127.635 0) (mirror x) (unit 1)
     (in_bom yes) (on_board yes)
-    (property "Reference" "Q?" (id 0) (at 243.205 128.905 0)
+    (property "Reference" "Q2" (id 0) (at 243.205 128.905 0)
       (effects (font (size 1.27 1.27)) (justify left))
     )
@@
   (symbol (lib_id "easyeda2kicad:47kΩ 0402 50V") (at 122.555 113.03 0) (unit 1)
     (in_bom yes) (on_board yes) (fields_autoplaced)
-    (property "Reference" "R?" (id 0) (at 122.555 107.315 0))
+    (property "Reference" "R6" (id 0) (at 122.555 107.315 0))
     (property "Value" "47kΩ 0402 50V" (id 1) (at 122.555 109.855 0))
     (property "Footprint" "easyeda2kicad:R0402" (id 2) (at 122.555 120.65 0)
@@
   (symbol (lib_id "easyeda2kicad:CP2102-GMR") (at 172.085 85.725 0) (unit 1)
     (in_bom yes) (on_board yes) (fields_autoplaced)
-    (property "Reference" "U?" (id 0) (at 198.12 71.5262 0))
+    (property "Reference" "U2" (id 0) (at 198.12 71.5262 0))
     (property "Value" "CP2102-GMR" (id 1) (at 198.12 74.0662 0))
     (property "Footprint" "easyeda2kicad:WQFN-28_L5.0-W5.0-P0.50-BL-EP3.2" (id 2) (at 172.085 116.205 0)
@@
   (symbol (lib_id "easyeda2kicad: 6.3V 10uF X5R ±20% 0402") (at 135.89 97.155 90) (unit 1)
     (in_bom yes) (on_board yes) (fields_autoplaced)
-    (property "Reference" "C?" (id 0) (at 139.7 95.8849 90)
+    (property "Reference" "C4" (id 0) (at 139.7 95.8849 90)
       (effects (font (size 1.27 1.27)) (justify right))
     )
@@
   (symbol (lib_id "power:GND") (at 149.225 83.185 270) (unit 1)
     (in_bom yes) (on_board yes) (fields_autoplaced)
-    (property "Reference" "#PWR?" (id 0) (at 142.875 83.185 0)
+    (property "Reference" "#PWR025" (id 0) (at 142.875 83.185 0)
       (effects (font (size 1.27 1.27)) hide)
     )
@@
   (symbol (lib_id "power:+3.3V") (at 149.225 93.345 90) (unit 1)
     (in_bom yes) (on_board yes) (fields_autoplaced)
-    (property "Reference" "#PWR?" (id 0) (at 153.035 93.345 0)
+    (property "Reference" "#PWR028" (id 0) (at 153.035 93.345 0)
       (effects (font (size 1.27 1.27)) hide)
     )
@@
   (symbol (lib_id "power:+3.3V") (at 149.225 90.805 90) (unit 1)
     (in_bom yes) (on_board yes) (fields_autoplaced)
-    (property "Reference" "#PWR?" (id 0) (at 153.035 90.805 0)
-      (effects (font (size 1.27 1.27)) hide)
-    )
+    (property "Reference" "#PWR026" (id 0) (at 153.035 90.805 0)
+      (effects (font (size 1.27 1.27)) hide)
+    )
