File: Hardware/cp2102.kicad_sch (KiCad schematic)
At the start: 12 parts, among them Q1 SS8050, Q2 SS8050, U2 CP2102-GMR

Commit message: V2 Board
Parts:
- removed R9: 22kΩ 0402 50V, easyeda2kicad:R0402, symbol easyeda2kicad:22kΩ 0402 50V
- renumbered C4 to C1, C5 to C2, R10 to R1, R7 to R2, R6 to R3, R8 to R5
Changed lines of the file:
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@@
   (junction (at 65.405 62.865) (diameter 0) (color 0 0 0 0)
-  )
-  (junction (at 127.635 113.03) (diameter 0) (color 0 0 0 0)
   )
   (no_connect (at 174.625 108.585))
@@
   (symbol (lib_id "easyeda2kicad:10kΩ 0402 50V") (at 229.235 113.665 0) (unit 1)
     (in_bom yes) (on_board yes) (fields_autoplaced)
-    (property "Reference" "R8" (id 0) (at 229.235 107.315 0))
+    (property "Reference" "R5" (id 0) (at 229.235 107.315 0))
     (property "Value" "10kΩ 0402 50V" (id 1) (at 229.235 109.855 0))
     (property "Footprint" "easyeda2kicad:R0402" (id 2) (at 229.235 121.285 0)
@@
   (symbol (lib_id "easyeda2kicad:25V 1uF X5R ±10% 0402") (at 132.08 118.11 90) (unit 1)
     (in_bom yes) (on_board yes) (fields_autoplaced)
-    (property "Reference" "C5" (id 0) (at 135.89 116.8399 90)
+    (property "Reference" "C2" (id 0) (at 135.89 116.8399 90)
       (effects (font (size 1.27 1.27)) (justify right))
     )
@@
   (symbol (lib_id "power:+3.3V") (at 167.005 118.745 180) (unit 1)
     (in_bom yes) (on_board yes) (fields_autoplaced)
-    (property "Reference" "#PWR031" (id 0) (at 167.005 114.935 0)
+    (property "Reference" "#PWR032" (id 0) (at 167.005 114.935 0)
       (effects (font (size 1.27 1.27)) hide)
     )
@@
     (pin "2")
     (pin "3")
-  )
-  (symbol (lib_id "easyeda2kicad:22kΩ 0402 50V") (at 127.635 118.11 90) (unit 1)
-    (in_bom yes) (on_board yes)
-    (property "Reference" "R9" (id 0) (at 123.19 116.84 90)
-      (effects (font (size 1.27 1.27)) (justify right))
-    )
-    (property "Value" "22kΩ 0402 50V" (id 1) (at 110.49 119.38 90)
-      (effects (font (size 1.27 1.27)) (justify right))
-    )
-    (property "Footprint" "easyeda2kicad:R0402" (id 2) (at 135.255 118.11 0)
-      (effects (font (size 1.27 1.27)) hide)
-    )
-    (property "Datasheet" "https://lcsc.com/product-detail/Chip-Resistor-Surface-Mount-UniOhm_22KR-2202-1_C25768.html" (id 3) (at 137.795 118.11 0)
-      (effects (font (size 1.27 1.27)) hide)
-    )
-    (property "Manufacturer" "UNI-ROYAL(厚声)" (id 4) (at 140.335 118.11 0)
-      (effects (font (size 1.27 1.27)) hide)
-    )
-    (property "LCSC Part" "C25768" (id 5) (at 142.875 118.11 0)
-      (effects (font (size 1.27 1.27)) hide)
-    )
-    (property "JLC Part" "Basic Part" (id 6) (at 145.415 118.11 0)
-      (effects (font (size 1.27 1.27)) hide)
-    )
-    (pin "1")
-    (pin "2")
   )
   (symbol (lib_id "easyeda2kicad:SRV05-4-P-T7 TVS") (at 76.835 90.17 270) (unit 1)
@@
     (pin "6")
   )
-  (symbol (lib_id "power:GND") (at 127.635 123.19 0) (unit 1)
-    (in_bom yes) (on_board yes) (fields_autoplaced)
-    (property "Reference" "#PWR032" (id 0) (at 127.635 129.54 0)
-      (effects (font (size 1.27 1.27)) hide)
-    )
-    (property "Value" "GND" (id 1) (at 127.635 128.27 0))
-    (property "Footprint" "" (id 2) (at 127.635 123.19 0)
-      (effects (font (size 1.27 1.27)) hide)
-    )
-    (property "Datasheet" "" (id 3) (at 127.635 123.19 0)
-      (effects (font (size 1.27 1.27)) hide)
-    )
-    (pin "1")
-  )
   (symbol (lib_id "easyeda2kicad:USB Micro B 1.8A") (at 40.005 62.865 0) (unit 1)
     (in_bom yes) (on_board yes) (fields_autoplaced)
@@
   (symbol (lib_id "power:GND") (at 27.305 62.865 270) (unit 1)
     (in_bom yes) (on_board yes) (fields_autoplaced)
-    (property "Reference" "#PWR022" (id 0) (at 20.955 62.865 0)
+    (property "Reference" "#PWR023" (id 0) (at 20.955 62.865 0)
       (effects (font (size 1.27 1.27)) hide)
     )
@@
   (symbol (lib_id "power:GND") (at 50.165 67.945 90) (unit 1)
     (in_bom yes) (on_board yes) (fields_autoplaced)
-    (property "Reference" "#PWR024" (id 0) (at 56.515 67.945 0)
+    (property "Reference" "#PWR025" (id 0) (at 56.515 67.945 0)
       (effects (font (size 1.27 1.27)) hide)
     )
@@
   (symbol (lib_id "easyeda2kicad:1kΩ 0402 50V") (at 167.005 113.665 90) (unit 1)
     (in_bom yes) (on_board yes) (fields_autoplaced)
-    (property "Reference" "R7" (id 0) (at 168.91 112.3949 90)
+    (property "Reference" "R2" (id 0) (at 168.91 112.3949 90)
       (effects (font (size 1.27 1.27)) (justify right))
     )
@@
   (symbol (lib_id "power:GND") (at 161.925 62.865 180) (unit 1)
     (in_bom yes) (on_board yes) (fields_autoplaced)
-    (property "Reference" "#PWR023" (id 0) (at 161.925 56.515 0)
+    (property "Reference" "#PWR024" (id 0) (at 161.925 56.515 0)
       (effects (font (size 1.27 1.27)) hide)
     )
@@
   (symbol (lib_id "easyeda2kicad:10kΩ 0402 50V") (at 229.235 127.635 0) (unit 1)
     (in_bom yes) (on_board yes) (fields_autoplaced)
-    (property "Reference" "R10" (id 0) (at 229.235 121.285 0))
+    (property "Reference" "R1" (id 0) (at 229.235 121.285 0))
     (property "Value" "10kΩ 0402 50V" (id 1) (at 229.235 123.825 0))
     (property "Footprint" "easyeda2kicad:R0402" (id 2) (at 229.235 135.255 0)
@@
   (symbol (lib_id "power:GND") (at 75.565 106.68 0) (unit 1)
     (in_bom yes) (on_board yes) (fields_autoplaced)
-    (property "Reference" "#PWR030" (id 0) (at 75.565 113.03 0)
+    (property "Reference" "#PWR031" (id 0) (at 75.565 113.03 0)
       (effects (font (size 1.27 1.27)) hide)
     )
@@
   (symbol (lib_id "power:GND") (at 135.89 100.965 0) (unit 1)
     (in_bom yes) (on_board yes) (fields_autoplaced)
-    (property "Reference" "#PWR029" (id 0) (at 135.89 107.315 0)
+    (property "Reference" "#PWR030" (id 0) (at 135.89 107.315 0)
       (effects (font (size 1.27 1.27)) hide)
     )
@@
   (symbol (lib_id "power:+3.3V") (at 135.89 93.345 0) (unit 1)
     (in_bom yes) (on_board yes)
-    (property "Reference" "#PWR027" (id 0) (at 135.89 97.155 0)
+    (property "Reference" "#PWR028" (id 0) (at 135.89 97.155 0)
       (effects (font (size 1.27 1.27)) hide)
     )
@@
   (symbol (lib_id "easyeda2kicad:47kΩ 0402 50V") (at 122.555 113.03 0) (unit 1)
     (in_bom yes) (on_board yes) (fields_autoplaced)
-    (property "Reference" "R6" (id 0) (at 122.555 107.315 0))
+    (property "Reference" "R3" (id 0) (at 122.555 107.315 0))
     (property "Value" "47kΩ 0402 50V" (id 1) (at 122.555 109.855 0))
     (property "Footprint" "easyeda2kicad:R0402" (id 2) (at 122.555 120.65 0)
@@
   (symbol (lib_id "easyeda2kicad: 6.3V 10uF X5R ±20% 0402") (at 135.89 97.155 90) (unit 1)
     (in_bom yes) (on_board yes) (fields_autoplaced)
-    (property "Reference" "C4" (id 0) (at 139.7 95.8849 90)
+    (property "Reference" "C1" (id 0) (at 139.7 95.8849 90)
       (effects (font (size 1.27 1.27)) (justify right))
     )
@@
   (symbol (lib_id "power:GND") (at 149.225 83.185 270) (unit 1)
     (in_bom yes) (on_board yes) (fields_autoplaced)
-    (property "Reference" "#PWR025" (id 0) (at 142.875 83.185 0)
+    (property "Reference" "#PWR026" (id 0) (at 142.875 83.185 0)
       (effects (font (size 1.27 1.27)) hide)
     )
@@
   (symbol (lib_id "power:+3.3V") (at 149.225 93.345 90) (unit 1)
     (in_bom yes) (on_board yes) (fields_autoplaced)
-    (property "Reference" "#PWR028" (id 0) (at 153.035 93.345 0)
+    (property "Reference" "#PWR029" (id 0) (at 153.035 93.345 0)
       (effects (font (size 1.27 1.27)) hide)
     )
@@
   (symbol (lib_id "power:+3.3V") (at 149.225 90.805 90) (unit 1)
     (in_bom yes) (on_board yes) (fields_autoplaced)
-    (property "Reference" "#PWR026" (id 0) (at 153.035 90.805 0)
-      (effects (font (size 1.27 1.27)) hide)
-    )
+    (property "Reference" "#PWR027" (id 0) (at 153.035 90.805 0)
+      (effects (font (size 1.27 1.27)) hide)
+    )
