File: Hardware/3V3.kicad_sch (KiCad schematic)
At the start: 12 parts, among them U5 TPS63020DSJR

Commit message: V2 Board
Parts:
- renumbered C13 to C10, C14 to C12, C8 to C3, C15 to C5, C12 to C6, C9 to C7, C10 to C9, R14 to R8, R15 to R9, U5 to U4
Changed lines of the file:
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@@
   (symbol (lib_id "easyeda2kicad: 6.3V 10uF X5R ±20% 0402") (at 170.942 85.852 90) (unit 1)
     (in_bom yes) (on_board yes) (fields_autoplaced)
-    (property "Reference" "C10" (id 0) (at 174.244 84.5819 90)
+    (property "Reference" "C9" (id 0) (at 174.244 84.5819 90)
       (effects (font (size 1.27 1.27)) (justify right))
     )
@@
   (symbol (lib_id "easyeda2kicad:180kΩ 0603 75V") (at 87.376 97.282 90) (unit 1)
     (in_bom yes) (on_board yes) (fields_autoplaced)
-    (property "Reference" "R15" (id 0) (at 89.916 96.0119 90)
+    (property "Reference" "R9" (id 0) (at 89.916 96.0119 90)
       (effects (font (size 1.27 1.27)) (justify right))
     )
@@
   (symbol (lib_id "easyeda2kicad:TPS63020DSJR") (at 128.27 84.582 0) (unit 1)
     (in_bom yes) (on_board yes) (fields_autoplaced)
-    (property "Reference" "U5" (id 0) (at 128.27 66.167 0))
+    (property "Reference" "U4" (id 0) (at 128.27 66.167 0))
     (property "Value" "TPS63020DSJR" (id 1) (at 128.27 68.707 0))
     (property "Footprint" "easyeda2kicad:VSON-14_L4.0-W3.0-P0.50-BL-EP_TI_DSJ" (id 2) (at 128.27 104.902 0)
@@
   (symbol (lib_id "easyeda2kicad:6.3V 22uF X5R ±20% 0603") (at 57.404 87.122 90) (unit 1)
     (in_bom yes) (on_board yes) (fields_autoplaced)
-    (property "Reference" "C13" (id 0) (at 60.706 85.8519 90)
+    (property "Reference" "C10" (id 0) (at 60.706 85.8519 90)
       (effects (font (size 1.27 1.27)) (justify right))
     )
@@
   (symbol (lib_id "easyeda2kicad:6.3V 22uF X5R ±20% 0603") (at 78.232 87.122 90) (unit 1)
     (in_bom yes) (on_board yes) (fields_autoplaced)
-    (property "Reference" "C15" (id 0) (at 81.534 85.8519 90)
+    (property "Reference" "C5" (id 0) (at 81.534 85.8519 90)
       (effects (font (size 1.27 1.27)) (justify right))
     )
@@
   (symbol (lib_id "easyeda2kicad:16V 100nF X7R ±10% 0402") (at 156.21 64.262 180) (unit 1)
     (in_bom yes) (on_board yes) (fields_autoplaced)
-    (property "Reference" "C8" (id 0) (at 156.21 57.277 0))
+    (property "Reference" "C3" (id 0) (at 156.21 57.277 0))
     (property "Value" "16V 100nF X7R ±10% 0402" (id 1) (at 156.21 59.817 0))
     (property "Footprint" "easyeda2kicad:C0402_NEW" (id 2) (at 156.21 56.642 0)
@@
   (symbol (lib_id "easyeda2kicad:1MΩ 0402 50V") (at 87.376 87.122 90) (unit 1)
     (in_bom yes) (on_board yes) (fields_autoplaced)
-    (property "Reference" "R14" (id 0) (at 89.916 85.8519 90)
+    (property "Reference" "R8" (id 0) (at 89.916 85.8519 90)
       (effects (font (size 1.27 1.27)) (justify right))
     )
@@
   (symbol (lib_id "easyeda2kicad:6.3V 22uF X5R ±20% 0603") (at 67.818 87.122 90) (unit 1)
     (in_bom yes) (on_board yes) (fields_autoplaced)
-    (property "Reference" "C14" (id 0) (at 71.12 85.8519 90)
+    (property "Reference" "C12" (id 0) (at 71.12 85.8519 90)
       (effects (font (size 1.27 1.27)) (justify right))
     )
@@
   (symbol (lib_id "easyeda2kicad: 6.3V 10uF X5R ±20% 0402") (at 160.528 85.852 90) (unit 1)
     (in_bom yes) (on_board yes) (fields_autoplaced)
-    (property "Reference" "C9" (id 0) (at 163.83 84.5819 90)
+    (property "Reference" "C7" (id 0) (at 163.83 84.5819 90)
       (effects (font (size 1.27 1.27)) (justify right))
     )
@@
   (symbol (lib_id "easyeda2kicad:6.3V 22uF X5R ±20% 0603") (at 46.99 87.122 90) (unit 1)
     (in_bom yes) (on_board yes) (fields_autoplaced)
-    (property "Reference" "C12" (id 0) (at 50.292 85.8519 90)
-      (effects (font (size 1.27 1.27)) (justify right))
-    )
+    (property "Reference" "C6" (id 0) (at 50.292 85.8519 90)
+      (effects (font (size 1.27 1.27)) (justify right))
+    )

Commit message: PCB V2
Parts:
- removed C10, C12, C5, C6: 22uF, easyeda2kicad:C0603, symbol easyeda2kicad:6.3V 22uF X5R ±20% 0603
- removed R8: 1MΩ 0402 50V, easyeda2kicad:R0402, symbol easyeda2kicad:1MΩ 0402 50V
- removed R9: 180kΩ 0603 75V, easyeda2kicad:R0603, symbol easyeda2kicad:180kΩ 0603 75V
- added C13: 22uF, easyeda2kicad:C0603, symbol easyeda2kicad:6.3V 22uF X5R ±20% 0603
- added C22: 10uF, easyeda2kicad:C0402, symbol easyeda2kicad: 6.3V 10uF X5R ±20% 0402
- added C23: 100uF, easyeda2kicad:CAP-SMD_L3.5-W2.8, symbol easyeda2kicad:100uF 6.3V Tantal 3528
- added C24: 100nF, easyeda2kicad:C0402_NEW, symbol easyeda2kicad:16V 100nF X7R ±10% 0402
- added D11, D12: SS14, easyeda2kicad:SMA_L4.2-W2.6-LS5.3-RD, symbol easyeda2kicad:SS14
- added L2 (x2): 120Ω 3A, easyeda2kicad:L1206, symbol easyeda2kicad:120Ω 3A
- added R2: 100kΩ 0402 50V, easyeda2kicad:R0402, symbol easyeda2kicad:100kΩ 0402 50V
- added R8: 18kΩ 0402 50V, easyeda2kicad:R0402, symbol easyeda2kicad:18kΩ 0402 50V
- renumbered C7 to C10, C9 to C11, C11 to C12, L1 to L4
Connections:
- net GND: now also C13.1, C22.1, C23.2, C24.1, R8.1
- net Vout: now also C24.2, L2.1; no longer U4.4 (VOUT), U4.5 (VOUT)
- net at U4.3 (FB): now also R2.1, R8.2
- net Vin: no longer names the net of C10.2, C11.2, U4.10 (VIN), U4.11 (VIN)
- net Vin: now also L2.1; no longer C12.2
- new net: C12.2, D11.1 (K), D12.1 (K), L2.2
- new net: C13.2, C22.2, C23.1, L2.2, R2.2, U4.4 (VOUT), U4.5 (VOUT)
- new net VBat: D12.2 (A)
- new net VUSB: D11.2 (A)
Other:
- moved on the sheet: C10, C11, C12, C3, L4, U4
