File: Hardware/audio_amplifier.kicad_sch (KiCad schematic)
At the start: 8 parts, among them U7 PAM8303DBSC

Commit message: V2 Board
Parts:
- renumbered C17 to C16, C21 to C17, C20 to C18, C18 to C19, C19 to C20, R17 to R14, R18 to R15, U7 to U6
Changed lines of the file:
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@@
   (symbol (lib_id "easyeda2kicad:25V 1uF X5R ±10% 0402") (at 33.02 89.662 90) (unit 1)
     (in_bom yes) (on_board yes) (fields_autoplaced)
-    (property "Reference" "C18" (id 0) (at 36.322 88.3919 90)
+    (property "Reference" "C19" (id 0) (at 36.322 88.3919 90)
       (effects (font (size 1.27 1.27)) (justify right))
     )
@@
   (symbol (lib_id "power:GND") (at 110.744 73.66 90) (unit 1)
     (in_bom yes) (on_board yes) (fields_autoplaced)
-    (property "Reference" "#PWR066" (id 0) (at 117.094 73.66 0)
+    (property "Reference" "#PWR070" (id 0) (at 117.094 73.66 0)
       (effects (font (size 1.27 1.27)) hide)
     )
@@
   (symbol (lib_id "easyeda2kicad:100uF 6.3V Tantal 3528") (at 33.02 112.522 90) (unit 1)
     (in_bom yes) (on_board yes) (fields_autoplaced)
-    (property "Reference" "C21" (id 0) (at 36.83 110.6169 90)
+    (property "Reference" "C17" (id 0) (at 36.83 110.6169 90)
       (effects (font (size 1.27 1.27)) (justify right))
     )
@@
   (symbol (lib_id "power:GND") (at 85.344 97.282 0) (unit 1)
     (in_bom yes) (on_board yes) (fields_autoplaced)
-    (property "Reference" "#PWR070" (id 0) (at 85.344 103.632 0)
+    (property "Reference" "#PWR072" (id 0) (at 85.344 103.632 0)
       (effects (font (size 1.27 1.27)) hide)
     )
@@
   (symbol (lib_id "easyeda2kicad: 50V 15nF X7R ±10% 0603") (at 110.744 93.472 90) (unit 1)
     (in_bom yes) (on_board yes) (fields_autoplaced)
-    (property "Reference" "C20" (id 0) (at 114.3 92.2019 90)
+    (property "Reference" "C18" (id 0) (at 114.3 92.2019 90)
       (effects (font (size 1.27 1.27)) (justify right))
     )
@@
   (symbol (lib_id "easyeda2kicad: 50V 15nF X7R ±10% 0603") (at 85.344 93.472 90) (unit 1)
     (in_bom yes) (on_board yes) (fields_autoplaced)
-    (property "Reference" "C19" (id 0) (at 88.9 92.2019 90)
+    (property "Reference" "C20" (id 0) (at 88.9 92.2019 90)
       (effects (font (size 1.27 1.27)) (justify right))
     )
@@
   (symbol (lib_id "power:GND") (at 33.02 116.332 0) (unit 1)
     (in_bom yes) (on_board yes) (fields_autoplaced)
-    (property "Reference" "#PWR072" (id 0) (at 33.02 122.682 0)
+    (property "Reference" "#PWR073" (id 0) (at 33.02 122.682 0)
       (effects (font (size 1.27 1.27)) hide)
     )
@@
   (symbol (lib_id "power:GND") (at 33.02 94.742 0) (unit 1)
     (in_bom yes) (on_board yes) (fields_autoplaced)
-    (property "Reference" "#PWR069" (id 0) (at 33.02 101.092 0)
+    (property "Reference" "#PWR071" (id 0) (at 33.02 101.092 0)
       (effects (font (size 1.27 1.27)) hide)
     )
@@
   (symbol (lib_id "easyeda2kicad:25V 1uF X5R ±10% 0402") (at 33.274 64.77 90) (unit 1)
     (in_bom yes) (on_board yes) (fields_autoplaced)
-    (property "Reference" "C17" (id 0) (at 36.576 63.4999 90)
+    (property "Reference" "C16" (id 0) (at 36.576 63.4999 90)
       (effects (font (size 1.27 1.27)) (justify right))
     )
@@
   (symbol (lib_id "power:GND") (at 33.274 69.85 0) (unit 1)
     (in_bom yes) (on_board yes) (fields_autoplaced)
-    (property "Reference" "#PWR064" (id 0) (at 33.274 76.2 0)
+    (property "Reference" "#PWR069" (id 0) (at 33.274 76.2 0)
       (effects (font (size 1.27 1.27)) hide)
     )
@@
   (symbol (lib_id "easyeda2kicad:PAM8303DBSC") (at 98.044 74.93 0) (unit 1)
     (in_bom yes) (on_board yes) (fields_autoplaced)
-    (property "Reference" "U7" (id 0) (at 98.044 63.5 0))
+    (property "Reference" "U6" (id 0) (at 98.044 63.5 0))
     (property "Value" "PAM8303DBSC" (id 1) (at 98.044 66.04 0))
     (property "Footprint" "easyeda2kicad:MSOP-8_L3.0-W3.0-P0.65-LS5.0-BL" (id 2) (at 98.044 86.36 0)
@@
   (symbol (lib_id "easyeda2kicad:150kΩ 0402 50V") (at 110.744 84.582 90) (unit 1)
     (in_bom yes) (on_board yes) (fields_autoplaced)
-    (property "Reference" "R18" (id 0) (at 113.03 83.3119 90)
+    (property "Reference" "R15" (id 0) (at 113.03 83.3119 90)
       (effects (font (size 1.27 1.27)) (justify right))
     )
@@
   (symbol (lib_id "easyeda2kicad:150kΩ 0402 50V") (at 85.344 84.582 90) (unit 1)
     (in_bom yes) (on_board yes) (fields_autoplaced)
-    (property "Reference" "R17" (id 0) (at 87.63 83.3119 90)
-      (effects (font (size 1.27 1.27)) (justify right))
-    )
+    (property "Reference" "R14" (id 0) (at 87.63 83.3119 90)
+      (effects (font (size 1.27 1.27)) (justify right))
+    )

Commit message: PCB V2
Parts:
- removed C16: 25V 1uF X5R ±10% 0402, easyeda2kicad:C0402, symbol easyeda2kicad:25V 1uF X5R ±10% 0402
- added C27: 100uF 6.3V Tantal 3528, easyeda2kicad:CAP-SMD_L3.5-W2.8, symbol easyeda2kicad:100uF 6.3V Tantal 3528
- added C28, C30: 16V 100nF X7R ±10% 0402, easyeda2kicad:C0402_NEW, symbol easyeda2kicad:16V 100nF X7R ±10% 0402
- added C31: 25V 1uF X5R ±10% 0402, easyeda2kicad:C0402, symbol easyeda2kicad:25V 1uF X5R ±10% 0402
- added L2: 120Ω 3A, easyeda2kicad:L1206, symbol easyeda2kicad:120Ω 3A
Connections:
- net GND: now also C27.2, C28.1, C30.1, C31.1
- net Vin: now also L2.1; no longer C19.2, U6.2 (PVDD), U6.3 (VDD)
- new net: C19.2, C27.1, C28.2, C30.2, C31.2, L2.2, U6.2 (PVDD), U6.3 (VDD)
Other:
- moved on the sheet: C17, C19
