File: Hardware/bms.kicad_sch (KiCad schematic)
At the start: 10 parts

Commit message: New pcb
Parts:
- removed CN?: B2B-PH-K-S(LF)(SN), easyeda2kicad:CONN-TH_B2B-PH-K-S, symbol easyeda2kicad:B2B-PH-K-S(LF)(SN)
- gave numbers to parts that had none: 9
Connections:
- net BAT renamed BAT+
Changed lines of the file:
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@@
     (effects (font (size 1.27 1.27)) (justify left bottom))
-  )
-  (label "BAT+" (at 234.95 63.5 180)
-    (effects (font (size 1.27 1.27)) (justify right bottom))
   )
   (label "Vin" (at 37.465 47.625 0)
     (effects (font (size 1.27 1.27)) (justify left bottom))
   )
+  (label "BAT-" (at 37.465 52.578 0)
+    (effects (font (size 1.27 1.27)) (justify left bottom))
+  )
   (label "BAT+" (at 37.465 50.165 0)
     (effects (font (size 1.27 1.27)) (justify left bottom))
@@
   (label "BAT+" (at 189.865 55.88 0)
     (effects (font (size 1.27 1.27)) (justify left bottom))
-  )
-  (label "BAT-" (at 234.95 68.58 180)
-    (effects (font (size 1.27 1.27)) (justify right bottom))
   )
   (label "BAT+" (at 86.995 78.74 180)
@@
     (effects (font (size 1.27 1.27)) (justify right))
   )
-  (hierarchical_label "BAT" (shape output) (at 37.465 50.165 180)
+  (hierarchical_label "BAT+" (shape output) (at 37.465 50.165 180)
     (effects (font (size 1.27 1.27)) (justify right))
   )
+  (hierarchical_label "BAT-" (shape output) (at 37.465 52.578 180)
+    (effects (font (size 1.27 1.27)) (justify right))
+  )
   (symbol (lib_id "power:GND") (at 67.31 87.63 0) (unit 1)
     (in_bom yes) (on_board yes) (fields_autoplaced)
-    (property "Reference" "#PWR?" (id 0) (at 67.31 93.98 0)
+    (property "Reference" "#PWR037" (id 0) (at 67.31 93.98 0)
       (effects (font (size 1.27 1.27)) hide)
     )
@@
   (symbol (lib_id "easyeda2kicad:25V 1uF X5R ±10% 0402") (at 67.31 82.55 90) (unit 1)
     (in_bom yes) (on_board yes) (fields_autoplaced)
-    (property "Reference" "C?" (id 0) (at 70.485 81.2799 90)
+    (property "Reference" "C7" (id 0) (at 70.485 81.2799 90)
       (effects (font (size 1.27 1.27)) (justify right))
     )
@@
     (pin "2")
   )
-  (symbol (lib_id "easyeda2kicad:B2B-PH-K-S(LF)(SN)") (at 241.3 66.04 180) (unit 1)
-    (in_bom yes) (on_board yes) (fields_autoplaced)
-    (property "Reference" "CN?" (id 0) (at 248.92 64.7699 0)
-      (effects (font (size 1.27 1.27)) (justify right))
-    )
-    (property "Value" "B2B-PH-K-S(LF)(SN)" (id 1) (at 248.92 67.3099 0)
-      (effects (font (size 1.27 1.27)) (justify right))
-    )
-    (property "Footprint" "easyeda2kicad:CONN-TH_B2B-PH-K-S" (id 2) (at 241.3 55.88 0)
-      (effects (font (size 1.27 1.27)) hide)
-    )
-    (property "Datasheet" "https://lcsc.com/product-detail/PH-Connectors_JST_B2B-PH-K-S-LF-SN_B2B-PH-K-S-LF-SN_C131337.html" (id 3) (at 241.3 53.34 0)
-      (effects (font (size 1.27 1.27)) hide)
-    )
-    (property "Manufacturer" "JST" (id 4) (at 241.3 50.8 0)
-      (effects (font (size 1.27 1.27)) hide)
-    )
-    (property "LCSC Part" "C131337" (id 5) (at 241.3 48.26 0)
-      (effects (font (size 1.27 1.27)) hide)
-    )
-    (property "JLC Part" "Extended Part" (id 6) (at 241.3 45.72 0)
-      (effects (font (size 1.27 1.27)) hide)
-    )
-    (pin "1")
-    (pin "2")
-  )
   (symbol (lib_id "easyeda2kicad:2kΩ 0402 50V") (at 122.555 68.58 180) (unit 1)
     (in_bom yes) (on_board yes) (fields_autoplaced)
-    (property "Reference" "R?" (id 0) (at 122.555 62.865 0))
+    (property "Reference" "R13" (id 0) (at 122.555 62.865 0))
     (property "Value" "2kΩ 0402 50V" (id 1) (at 122.555 65.405 0))
     (property "Footprint" "easyeda2kicad:R0402" (id 2) (at 122.555 60.96 0)
@@
   (symbol (lib_id "power:GND") (at 86.995 73.66 270) (unit 1)
     (in_bom yes) (on_board yes) (fields_autoplaced)
-    (property "Reference" "#PWR?" (id 0) (at 80.645 73.66 0)
+    (property "Reference" "#PWR036" (id 0) (at 80.645 73.66 0)
       (effects (font (size 1.27 1.27)) hide)
     )
@@
   (symbol (lib_id "power:GND") (at 163.195 71.12 0) (unit 1)
     (in_bom yes) (on_board yes) (fields_autoplaced)
-    (property "Reference" "#PWR?" (id 0) (at 163.195 77.47 0)
+    (property "Reference" "#PWR035" (id 0) (at 163.195 77.47 0)
       (effects (font (size 1.27 1.27)) hide)
     )
@@
   (symbol (lib_id "easyeda2kicad:BRCL3130ME") (at 173.355 68.58 180) (unit 1)
     (in_bom yes) (on_board yes) (fields_autoplaced)
-    (property "Reference" "U?" (id 0) (at 173.355 58.42 0))
+    (property "Reference" "U3" (id 0) (at 173.355 58.42 0))
     (property "Value" "BRCL3130ME" (id 1) (at 173.355 60.96 0))
     (property "Footprint" "easyeda2kicad:SOT-23-5_L2.9-W1.6-P0.95-LS2.8-BL" (id 2) (at 173.355 58.42 0)
@@
   (symbol (lib_id "easyeda2kicad:Green LED 0603") (at 122.555 74.93 180) (unit 1)
     (in_bom yes) (on_board yes)
-    (property "Reference" "LED?" (id 0) (at 126.365 75.565 0))
+    (property "Reference" "LED2" (id 0) (at 126.365 75.565 0))
     (property "Value" "Green LED 0603" (id 1) (at 131.445 77.47 0))
     (property "Footprint" "easyeda2kicad:LED0603-R-RD" (id 2) (at 122.555 66.04 0)
@@
   (symbol (lib_id "easyeda2kicad:TP4057") (at 102.235 73.66 0) (unit 1)
     (in_bom yes) (on_board yes) (fields_autoplaced)
-    (property "Reference" "U?" (id 0) (at 102.235 60.96 0))
+    (property "Reference" "U4" (id 0) (at 102.235 60.96 0))
     (property "Value" "TP4057" (id 1) (at 102.235 63.5 0))
     (property "Footprint" "easyeda2kicad:SOT-23-6_L2.9-W1.6-P0.95-LS2.8-BR" (id 2) (at 102.235 86.36 0)
@@
   (symbol (lib_id "easyeda2kicad:100Ω 0402 50V") (at 189.865 60.96 90) (unit 1)
     (in_bom yes) (on_board yes) (fields_autoplaced)
-    (property "Reference" "R?" (id 0) (at 191.77 59.6899 90)
+    (property "Reference" "R12" (id 0) (at 191.77 59.6899 90)
       (effects (font (size 1.27 1.27)) (justify right))
     )
@@
   (symbol (lib_id "easyeda2kicad:1kΩ 0402 50V") (at 64.77 53.34 90) (unit 1)
     (in_bom yes) (on_board yes) (fields_autoplaced)
-    (property "Reference" "R?" (id 0) (at 67.31 52.0699 90)
+    (property "Reference" "R11" (id 0) (at 67.31 52.0699 90)
       (effects (font (size 1.27 1.27)) (justify right))
     )
@@
   (symbol (lib_id "easyeda2kicad:Red LED 0603") (at 66.04 63.5 90) (unit 1)
     (in_bom yes) (on_board yes) (fields_autoplaced)
-    (property "Reference" "LED?" (id 0) (at 69.85 63.4999 90)
+    (property "Reference" "LED1" (id 0) (at 69.85 63.4999 90)
       (effects (font (size 1.27 1.27)) (justify right))
     )
@@
   (symbol (lib_id "power:GND") (at 127.635 68.58 90) (unit 1)
     (in_bom yes) (on_board yes) (fields_autoplaced)
-    (property "Reference" "#PWR?" (id 0) (at 133.985 68.58 0)
+    (property "Reference" "#PWR034" (id 0) (at 133.985 68.58 0)
       (effects (font (size 1.27 1.27)) hide)
     )
@@
   (symbol (lib_id "easyeda2kicad:25V 1uF X5R ±10% 0402") (at 189.865 71.12 90) (unit 1)
     (in_bom yes) (on_board yes) (fields_autoplaced)
-    (property "Reference" "C?" (id 0) (at 193.675 69.8499 90)
-      (effects (font (size 1.27 1.27)) (justify right))
-    )
+    (property "Reference" "C6" (id 0) (at 193.675 69.8499 90)
+      (effects (font (size 1.27 1.27)) (justify right))
+    )

Commit message: V2 Board
Parts:
- removed C6: 25V 1uF X5R ±10% 0402, easyeda2kicad:C0402, symbol easyeda2kicad:25V 1uF X5R ±10% 0402
- removed R12: 100Ω 0402 50V, easyeda2kicad:R0402, symbol easyeda2kicad:100Ω 0402 50V
- removed U3: BRCL3130ME, easyeda2kicad:SOT-23-5_L2.9-W1.6-P0.95-LS2.8-BL, symbol easyeda2kicad:BRCL3130ME
- renumbered C7 to C8, R13 to R4, R11 to R7, U4 to U1
Connections:
- no-connect marks 1 -> 0
Changed lines of the file:
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@@
 (kicad_sch (version 20211123) (generator eeschema)
   (paper "A4")
-  (junction (at 189.865 66.04) (diameter 0) (color 0 0 0 0)
-  )
   (junction (at 64.77 58.42) (diameter 0) (color 0 0 0 0)
   )
-  (junction (at 163.195 71.12) (diameter 0) (color 0 0 0 0)
-  )
-  (no_connect (at 183.515 71.12))
   (wire (pts (xy 127.635 73.66) (xy 139.7 73.66))
     (stroke (width 0) (type default) (color 0 0 0 0))
   )
-  (wire (pts (xy 186.69 68.58) (xy 186.69 76.2))
-    (stroke (width 0) (type default) (color 0 0 0 0))
-  )
   (wire (pts (xy 139.7 58.42) (xy 64.77 58.42))
     (stroke (width 0) (type default) (color 0 0 0 0))
   )
-  (wire (pts (xy 183.515 68.58) (xy 186.69 68.58))
-    (stroke (width 0) (type default) (color 0 0 0 0))
-  )
   (wire (pts (xy 139.7 73.66) (xy 139.7 58.42))
     (stroke (width 0) (type default) (color 0 0 0 0))
@@
     (stroke (width 0) (type default) (color 0 0 0 0))
   )
-  (wire (pts (xy 183.515 66.04) (xy 189.865 66.04))
-    (stroke (width 0) (type default) (color 0 0 0 0))
-  )
-  (wire (pts (xy 163.195 66.04) (xy 163.195 71.12))
-    (stroke (width 0) (type default) (color 0 0 0 0))
-  )
-  (wire (pts (xy 186.69 76.2) (xy 189.865 76.2))
-    (stroke (width 0) (type default) (color 0 0 0 0))
-  )
-  (label "BAT-" (at 189.865 76.2 0)
-    (effects (font (size 1.27 1.27)) (justify left bottom))
-  )
   (label "Vin" (at 67.31 77.47 0)
     (effects (font (size 1.27 1.27)) (justify left bottom))
@@
     (effects (font (size 1.27 1.27)) (justify left bottom))
   )
+  (label "BAT-" (at 34.798 59.944 0)
+    (effects (font (size 1.27 1.27)) (justify left bottom))
+  )
   (label "BAT+" (at 37.465 50.165 0)
     (effects (font (size 1.27 1.27)) (justify left bottom))
   )
   (label "Vin" (at 64.77 48.26 0)
-    (effects (font (size 1.27 1.27)) (justify left bottom))
-  )
-  (label "BAT+" (at 189.865 55.88 0)
     (effects (font (size 1.27 1.27)) (justify left bottom))
   )
@@
   (symbol (lib_id "easyeda2kicad:25V 1uF X5R ±10% 0402") (at 67.31 82.55 90) (unit 1)
     (in_bom yes) (on_board yes) (fields_autoplaced)
-    (property "Reference" "C7" (id 0) (at 70.485 81.2799 90)
+    (property "Reference" "C8" (id 0) (at 70.485 81.2799 90)
       (effects (font (size 1.27 1.27)) (justify right))
     )
@@
   (symbol (lib_id "easyeda2kicad:2kΩ 0402 50V") (at 122.555 68.58 180) (unit 1)
     (in_bom yes) (on_board yes) (fields_autoplaced)
-    (property "Reference" "R13" (id 0) (at 122.555 62.865 0))
+    (property "Reference" "R4" (id 0) (at 122.555 62.865 0))
     (property "Value" "2kΩ 0402 50V" (id 1) (at 122.555 65.405 0))
     (property "Footprint" "easyeda2kicad:R0402" (id 2) (at 122.555 60.96 0)
@@
     )
     (pin "1")
-  )
-  (symbol (lib_id "power:GND") (at 163.195 71.12 0) (unit 1)
-    (in_bom yes) (on_board yes) (fields_autoplaced)
-    (property "Reference" "#PWR035" (id 0) (at 163.195 77.47 0)
-      (effects (font (size 1.27 1.27)) hide)
-    )
-    (property "Value" "GND" (id 1) (at 163.195 76.2 0))
-    (property "Footprint" "" (id 2) (at 163.195 71.12 0)
-      (effects (font (size 1.27 1.27)) hide)
-    )
-    (property "Datasheet" "" (id 3) (at 163.195 71.12 0)
-      (effects (font (size 1.27 1.27)) hide)
-    )
-    (pin "1")
-  )
-  (symbol (lib_id "easyeda2kicad:BRCL3130ME") (at 173.355 68.58 180) (unit 1)
-    (in_bom yes) (on_board yes) (fields_autoplaced)
-    (property "Reference" "U3" (id 0) (at 173.355 58.42 0))
-    (property "Value" "BRCL3130ME" (id 1) (at 173.355 60.96 0))
-    (property "Footprint" "easyeda2kicad:SOT-23-5_L2.9-W1.6-P0.95-LS2.8-BL" (id 2) (at 173.355 58.42 0)
-      (effects (font (size 1.27 1.27)) hide)
-    )
-    (property "Datasheet" "https://lcsc.com/product-detail/PMIC-Battery-Management_BLUE-ROCKET-BRCL3130ME_C328560.html" (id 3) (at 173.355 55.88 0)
-      (effects (font (size 1.27 1.27)) hide)
-    )
-    (property "Manufacturer" "BLUE ROCKET(蓝箭)" (id 4) (at 173.355 53.34 0)
-      (effects (font (size 1.27 1.27)) hide)
-    )
-    (property "LCSC Part" "C328560" (id 5) (at 173.355 50.8 0)
-      (effects (font (size 1.27 1.27)) hide)
-    )
-    (property "JLC Part" "Extended Part" (id 6) (at 173.355 48.26 0)
-      (effects (font (size 1.27 1.27)) hide)
-    )
-    (pin "1")
-    (pin "2")
-    (pin "3")
-    (pin "4")
-    (pin "5")
   )
   (symbol (lib_id "easyeda2kicad:Green LED 0603") (at 122.555 74.93 180) (unit 1)
@@
   (symbol (lib_id "easyeda2kicad:TP4057") (at 102.235 73.66 0) (unit 1)
     (in_bom yes) (on_board yes) (fields_autoplaced)
-    (property "Reference" "U4" (id 0) (at 102.235 60.96 0))
+    (property "Reference" "U1" (id 0) (at 102.235 60.96 0))
     (property "Value" "TP4057" (id 1) (at 102.235 63.5 0))
     (property "Footprint" "easyeda2kicad:SOT-23-6_L2.9-W1.6-P0.95-LS2.8-BR" (id 2) (at 102.235 86.36 0)
@@
     (pin "6")
   )
-  (symbol (lib_id "easyeda2kicad:100Ω 0402 50V") (at 189.865 60.96 90) (unit 1)
-    (in_bom yes) (on_board yes) (fields_autoplaced)
-    (property "Reference" "R12" (id 0) (at 191.77 59.6899 90)
-      (effects (font (size 1.27 1.27)) (justify right))
-    )
-    (property "Value" "100Ω 0402 50V" (id 1) (at 191.77 62.2299 90)
-      (effects (font (size 1.27 1.27)) (justify right))
-    )
-    (property "Footprint" "easyeda2kicad:R0402" (id 2) (at 197.485 60.96 0)
-      (effects (font (size 1.27 1.27)) hide)
-    )
-    (property "Datasheet" "https://lcsc.com/product-detail/Chip-Resistor-Surface-Mount-UniOhm_100R-1000-1_C25076.html" (id 3) (at 200.025 60.96 0)
-      (effects (font (size 1.27 1.27)) hide)
-    )
-    (property "Manufacturer" "UNI-ROYAL(厚声)" (id 4) (at 202.565 60.96 0)
-      (effects (font (size 1.27 1.27)) hide)
-    )
-    (property "LCSC Part" "C25076" (id 5) (at 205.105 60.96 0)
-      (effects (font (size 1.27 1.27)) hide)
-    )
-    (property "JLC Part" "Basic Part" (id 6) (at 207.645 60.96 0)
-      (effects (font (size 1.27 1.27)) hide)
-    )
-    (pin "1")
-    (pin "2")
-  )
   (symbol (lib_id "easyeda2kicad:1kΩ 0402 50V") (at 64.77 53.34 90) (unit 1)
     (in_bom yes) (on_board yes) (fields_autoplaced)
-    (property "Reference" "R11" (id 0) (at 67.31 52.0699 90)
+    (property "Reference" "R7" (id 0) (at 67.31 52.0699 90)
       (effects (font (size 1.27 1.27)) (justify right))
     )
@@
     (pin "2")
   )
+  (symbol (lib_id "power:GND") (at 34.798 59.944 0) (unit 1)
+    (in_bom yes) (on_board yes) (fields_autoplaced)
+    (property "Reference" "#PWR034" (id 0) (at 34.798 66.294 0)
+      (effects (font (size 1.27 1.27)) hide)
+    )
+    (property "Value" "GND" (id 1) (at 34.798 64.77 0))
+    (property "Footprint" "" (id 2) (at 34.798 59.944 0)
+      (effects (font (size 1.27 1.27)) hide)
+    )
+    (property "Datasheet" "" (id 3) (at 34.798 59.944 0)
+      (effects (font (size 1.27 1.27)) hide)
+    )
+    (pin "1")
+  )
   (symbol (lib_id "power:GND") (at 127.635 68.58 90) (unit 1)
     (in_bom yes) (on_board yes) (fields_autoplaced)
-    (property "Reference" "#PWR034" (id 0) (at 133.985 68.58 0)
+    (property "Reference" "#PWR035" (id 0) (at 133.985 68.58 0)
       (effects (font (size 1.27 1.27)) hide)
     )
@@
     (pin "1")
   )
-  (symbol (lib_id "easyeda2kicad:25V 1uF X5R ±10% 0402") (at 189.865 71.12 90) (unit 1)
-    (in_bom yes) (on_board yes) (fields_autoplaced)
-    (property "Reference" "C6" (id 0) (at 193.675 69.8499 90)
-      (effects (font (size 1.27 1.27)) (justify right))
-    )
-    (property "Value" "25V 1uF X5R ±10% 0402" (id 1) (at 193.675 72.3899 90)
-      (effects (font (size 1.27 1.27)) (justify right))
-    )
-    (property "Footprint" "easyeda2kicad:C0402" (id 2) (at 197.485 71.12 0)
-      (effects (font (size 1.27 1.27)) hide)
-    )
-    (property "Datasheet" "https://lcsc.com/product-detail/Multilayer-Ceramic-Capacitors-MLCC-SMD-SMT_SAMSUNG_CL05A105KA5NQNC_1uF-105-10-25V_C52923.html" (id 3) (at 200.025 71.12 0)
-      (effects (font (size 1.27 1.27)) hide)
-    )
-    (property "Manufacturer" "SAMSUNG(三星)" (id 4) (at 202.565 71.12 0)
-      (effects (font (size 1.27 1.27)) hide)
-    )
-    (property "LCSC Part" "C52923" (id 5) (at 205.105 71.12 0)
-      (effects (font (size 1.27 1.27)) hide)
-    )
-    (property "JLC Part" "Basic Part" (id 6) (at 207.645 71.12 0)
-      (effects (font (size 1.27 1.27)) hide)
-    )
-    (pin "1")
-    (pin "2")
-  )
 )
