File: Hardware/esp32.kicad_sch (KiCad schematic)
At the start: 7 parts

Commit message: New pcb
Parts:
- removed LED?: Red LED 0603, easyeda2kicad:LED0603-R-RD, symbol easyeda2kicad:Red LED 0603
- removed R?: 1kΩ 0402 50V, easyeda2kicad:R0402, symbol easyeda2kicad:1kΩ 0402 50V
- gave numbers to parts that had none: 3
- renumbered C1 to C3, R1 to R5
Connections:
- net IO2: now reaches U1.24 (IO2)
- net IO5: now reaches U1.29 (IO5)
- no-connect marks 10 -> 9
Other:
- moved on the sheet: C1, C2, C3, R5, U1

Commit message: V2 Board
Parts:
- renumbered C3 to C13, C1 to C14, C2 to C15, R5 to R13, U1 to U5
Changed lines of the file:
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@@
   (symbol (lib_id "power:+3.3V") (at 69.215 85.598 90) (unit 1)
     (in_bom yes) (on_board yes) (fields_autoplaced)
-    (property "Reference" "#PWR019" (id 0) (at 73.025 85.598 0)
+    (property "Reference" "#PWR020" (id 0) (at 73.025 85.598 0)
       (effects (font (size 1.27 1.27)) hide)
     )
@@
   (symbol (lib_id "power:GND") (at 79.375 95.758 0) (unit 1)
     (in_bom yes) (on_board yes) (fields_autoplaced)
-    (property "Reference" "#PWR021" (id 0) (at 79.375 102.108 0)
+    (property "Reference" "#PWR022" (id 0) (at 79.375 102.108 0)
       (effects (font (size 1.27 1.27)) hide)
     )
@@
   (symbol (lib_id "power:GND") (at 156.21 55.118 90) (unit 1)
     (in_bom yes) (on_board yes) (fields_autoplaced)
-    (property "Reference" "#PWR016" (id 0) (at 162.56 55.118 0)
+    (property "Reference" "#PWR017" (id 0) (at 162.56 55.118 0)
       (effects (font (size 1.27 1.27)) hide)
     )
@@
   (symbol (lib_id "easyeda2kicad: 6.3V 10uF X5R ±20% 0402") (at 93.345 55.118 90) (unit 1)
     (in_bom yes) (on_board yes) (fields_autoplaced)
-    (property "Reference" "C1" (id 0) (at 96.52 53.8479 90)
+    (property "Reference" "C14" (id 0) (at 96.52 53.8479 90)
       (effects (font (size 1.27 1.27)) (justify right))
     )
@@
   (symbol (lib_id "power:+3.3V") (at 125.73 57.658 90) (unit 1)
     (in_bom yes) (on_board yes) (fields_autoplaced)
-    (property "Reference" "#PWR017" (id 0) (at 129.54 57.658 0)
+    (property "Reference" "#PWR018" (id 0) (at 129.54 57.658 0)
       (effects (font (size 1.27 1.27)) hide)
     )
@@
   (symbol (lib_id "easyeda2kicad:10kΩ 0402 50V") (at 74.295 85.598 0) (unit 1)
     (in_bom yes) (on_board yes) (fields_autoplaced)
-    (property "Reference" "R5" (id 0) (at 74.295 79.883 0))
+    (property "Reference" "R13" (id 0) (at 74.295 79.883 0))
     (property "Value" "10kΩ 0402 50V" (id 1) (at 74.295 82.423 0))
     (property "Footprint" "easyeda2kicad:R0402" (id 2) (at 74.295 93.218 0)
@@
   (symbol (lib_id "power:GND") (at 93.345 58.928 0) (unit 1)
     (in_bom yes) (on_board yes) (fields_autoplaced)
-    (property "Reference" "#PWR018" (id 0) (at 93.345 65.278 0)
+    (property "Reference" "#PWR019" (id 0) (at 93.345 65.278 0)
       (effects (font (size 1.27 1.27)) hide)
     )
@@
   (symbol (lib_id "easyeda2kicad:25V 1uF X5R ±10% 0402") (at 79.375 90.678 90) (unit 1)
     (in_bom yes) (on_board yes) (fields_autoplaced)
-    (property "Reference" "C3" (id 0) (at 83.185 89.4079 90)
+    (property "Reference" "C13" (id 0) (at 83.185 89.4079 90)
       (effects (font (size 1.27 1.27)) (justify right))
     )
@@
   (symbol (lib_id "easyeda2kicad:16V 100nF X7R ±10% 0402") (at 105.41 55.118 90) (unit 1)
     (in_bom yes) (on_board yes) (fields_autoplaced)
-    (property "Reference" "C2" (id 0) (at 109.22 53.8479 90)
+    (property "Reference" "C15" (id 0) (at 109.22 53.8479 90)
       (effects (font (size 1.27 1.27)) (justify right))
     )
@@
   (symbol (lib_id "power:GND") (at 125.73 90.678 270) (unit 1)
     (in_bom yes) (on_board yes) (fields_autoplaced)
-    (property "Reference" "#PWR020" (id 0) (at 119.38 90.678 0)
+    (property "Reference" "#PWR021" (id 0) (at 119.38 90.678 0)
       (effects (font (size 1.27 1.27)) hide)
     )
@@
   (symbol (lib_id "power:GND") (at 125.73 55.118 270) (unit 1)
     (in_bom yes) (on_board yes) (fields_autoplaced)
-    (property "Reference" "#PWR015" (id 0) (at 119.38 55.118 0)
+    (property "Reference" "#PWR016" (id 0) (at 119.38 55.118 0)
       (effects (font (size 1.27 1.27)) hide)
     )
@@
   (symbol (lib_id "power:+3.3V") (at 93.345 51.308 0) (unit 1)
     (in_bom yes) (on_board yes) (fields_autoplaced)
-    (property "Reference" "#PWR013" (id 0) (at 93.345 55.118 0)
+    (property "Reference" "#PWR014" (id 0) (at 93.345 55.118 0)
       (effects (font (size 1.27 1.27)) hide)
     )
@@
   (symbol (lib_id "power:GND") (at 156.21 52.578 90) (unit 1)
     (in_bom yes) (on_board yes) (fields_autoplaced)
-    (property "Reference" "#PWR014" (id 0) (at 162.56 52.578 0)
+    (property "Reference" "#PWR015" (id 0) (at 162.56 52.578 0)
       (effects (font (size 1.27 1.27)) hide)
     )
@@
   (symbol (lib_id "easyeda2kicad:ESP32-WROOM-32D(8MB)") (at 140.97 77.978 0) (unit 1)
     (in_bom yes) (on_board yes) (fields_autoplaced)
-    (property "Reference" "U1" (id 0) (at 140.97 46.228 0))
+    (property "Reference" "U5" (id 0) (at 140.97 46.228 0))
     (property "Value" "ESP32-WROOM-32D(8MB)" (id 1) (at 140.97 48.768 0))
     (property "Footprint" "easyeda2kicad:WIFIM-SMD_39P-L25.5-W18.0-P1.27" (id 2) (at 140.97 108.458 0)

Commit message: PCB V2
Parts:
- removed C13: 25V 1uF X5R ±10% 0402, easyeda2kicad:C0402, symbol easyeda2kicad:25V 1uF X5R ±10% 0402
- removed C15: 100nF, easyeda2kicad:C0402_NEW, symbol easyeda2kicad:16V 100nF X7R ±10% 0402
- added C1: 100nF, easyeda2kicad:C0402_NEW, symbol easyeda2kicad:16V 100nF X7R ±10% 0402
- added C15, C2, C4: 10uF, easyeda2kicad:C0402, symbol easyeda2kicad: 6.3V 10uF X5R ±20% 0402
- added L2: 120Ω 3A, easyeda2kicad:L1206, symbol easyeda2kicad:120Ω 3A
- added R1: 10kΩ 0402 50V, easyeda2kicad:R0402, symbol easyeda2kicad:10kΩ 0402 50V
Connections:
- net +3.3V: now also C15.2, C2.2, L2.1, R1.2; no longer U5.2 (VDD33)
- net ESP_EN: now also C4.2
- net ESP_IO0: now also R1.1
- net GND: now also C1.1, C15.1, C2.1, C4.1
- new net: C1.2, L2.2, U5.2 (VDD33)
Other:
- moved on the sheet: R13, U5
