File: Hardware/servo_extender.kicad_sch (KiCad schematic)
At the start: 6 parts, among them U6 PCA9685PW,118

Commit message: V2 Board
Parts:
- added H8, H9: Header 2.54 5P Female, easyeda2kicad:HDR-TH_5P-P2.54-V-F, symbol easyeda2kicad:Header 2.54 5P Female
- renumbered C16 to C21, H5 to H4, H7 to H5, H6 to H7, U6 to U7
Connections:
- net +3.3V: now also H8.2, H9.2
- net +BATT: now also H8.1, H9.1
- net GND: now also H8.5, H9.5
- net SCL: now also H8.4, H9.4
- net SDA: now also H8.3, H9.3

Commit message: PCB V2
Parts:
- removed C21: 6.3V 10uF X5R ±20% 0402, easyeda2kicad:C0402, symbol easyeda2kicad: 6.3V 10uF X5R ±20% 0402
- removed H4, H5, H7: 9P 2.54 Male Header, easyeda2kicad:HDR-TH_9P-P2.54-V-M, symbol easyeda2kicad:9P 2.54 Male Header
- added C16: 100nF, easyeda2kicad:C0402_NEW, symbol easyeda2kicad:16V 100nF X7R ±10% 0402
- added C21: 22uF, easyeda2kicad:C0603, symbol easyeda2kicad:6.3V 22uF X5R ±20% 0603
- added D1: SMF05CT1G, easyeda2kicad:SOT-363_L2.0-W1.3-P0.65-LS2.1-BR, symbol easyeda2kicad:SMF05CT1G
- added LED3: White Led 0603, easyeda2kicad:LED0603-R-RD_WHITE, symbol easyeda2kicad:White Led 0603
- added R17, R18: 10kΩ 0402 50V, easyeda2kicad:R0402, symbol easyeda2kicad:10kΩ 0402 50V
- added R4: 4.7kΩ 0402 50V, easyeda2kicad:R0402, symbol easyeda2kicad:4.7kΩ 0402 50V
Connections:
- net +3.3V: now also U7.1 (A0), U7.2 (A1), U7.3 (A2), U7.4 (A3), U7.5 (A4), C16.2, C21.2, D1.6, R17.1, R18.1, R4.2
- net +BATT: now also D1.1
- net GND: now also C16.1, C21.1, D1.2, LED3.2 (K); no longer U7.1 (A0), U7.2 (A1), U7.3 (A2), U7.4 (A3), U7.5 (A4)
- net SCL: now also D1.3, D1.4, R17.2
- net SDA: now also D1.5, R18.2
- new net: LED3.1 (A), R4.1
Other:
- added sheet Servo Connectors1 (servo.kicad_sch)
- moved on the sheet: H8, R16, U7
